Commit message: Add SLAM, Nav2, and autonomous exploration features
- Add auto_explorer.py for frontier-based autonomous exploration
- Add SLAM, localization, and navigation launch files
- Add Nav2 and EKF configuration files
- Add multiple simulation worlds (warehouse, office_maze, f1_circuit, etc.)
- Update robot URDF with sensors (LiDAR, camera, IMU)
- Remove old robot_controller package

Co-Authored-By: Claude Opus 4.5 <noreply@anthropic.com>

File: drobot_simulation/urdf/drobot.urdf.xacro (robot description, xacro)
@@ -13,5 +13,6 @@
   <xacro:property name="wheel_width" value="0.04"/>
   <xacro:property name="wheel_mass" value="0.2"/>
-  <xacro:property name="wheel_base" value="0.24"/>  <!-- 바퀴 간 거리 -->
+  <xacro:property name="wheel_base" value="0.24"/>  <!-- 좌우 바퀴 간 거리 -->
+  <xacro:property name="wheel_separation_length" value="0.20"/>  <!-- 앞뒤 바퀴 간 거리 -->
   <!-- 프로펠러 파라미터 -->
   <xacro:property name="prop_radius" value="0.08"/>
@@ -48,6 +49,6 @@
              izz="${m*r*r/2}"/>
   </xacro:macro>
-  <!-- 바퀴 매크로 -->
-  <xacro:macro name="wheel" params="prefix y_offset">
+  <!-- 바퀴 매크로 (4바퀴 지원) -->
+  <xacro:macro name="wheel" params="prefix x_offset y_offset">
     <link name="${prefix}_wheel">
       <visual>
@@ -73,5 +74,5 @@
       <parent link="base_link"/>
       <child link="${prefix}_wheel"/>
-      <origin xyz="0 ${y_offset} 0" rpy="0 0 0"/>
+      <origin xyz="${x_offset} ${y_offset} 0" rpy="0 0 0"/>
       <axis xyz="0 1 0"/>
       <dynamics damping="0.1" friction="0.1"/>
@@ -155,36 +156,12 @@
   </gazebo>
   <!-- ==================== -->
-  <!-- WHEELS (바퀴)        -->
-  <!-- ==================== -->
-  <xacro:wheel prefix="left" y_offset="${wheel_base/2}"/>
-  <xacro:wheel prefix="right" y_offset="${-wheel_base/2}"/>
-  <!-- 캐스터 휠 (보조 바퀴) -->
-  <link name="caster_wheel">
-    <visual>
-      <geometry>
-        <sphere radius="${wheel_radius * 0.5}"/>
-      </geometry>
-      <material name="gray"/>
-    </visual>
-    <collision>
-      <geometry>
-        <sphere radius="${wheel_radius * 0.5}"/>
-      </geometry>
-    </collision>
-    <inertial>
-      <mass value="0.1"/>
-      <inertia ixx="0.00001" ixy="0" ixz="0" iyy="0.00001" iyz="0" izz="0.00001"/>
-    </inertial>
-  </link>
-  <joint name="caster_joint" type="fixed">
-    <parent link="base_link"/>
-    <child link="caster_wheel"/>
-    <origin xyz="${-body_length/2 + 0.03} 0 ${-wheel_radius * 0.5}" rpy="0 0 0"/>
-  </joint>
-  <gazebo reference="caster_wheel">
-    <mu1>0.001</mu1>
-    <mu2>0.001</mu2>
-    <material>Gazebo/Grey</material>
-  </gazebo>
+  <!-- WHEELS (4바퀴 스키드 스티어) -->
+  <!-- ==================== -->
+  <!-- 앞바퀴 -->
+  <xacro:wheel prefix="front_left"  x_offset="${wheel_separation_length/2}"  y_offset="${wheel_base/2}"/>
+  <xacro:wheel prefix="front_right" x_offset="${wheel_separation_length/2}"  y_offset="${-wheel_base/2}"/>
+  <!-- 뒷바퀴 -->
+  <xacro:wheel prefix="rear_left"   x_offset="${-wheel_separation_length/2}" y_offset="${wheel_base/2}"/>
+  <xacro:wheel prefix="rear_right"  x_offset="${-wheel_separation_length/2}" y_offset="${-wheel_base/2}"/>
   <!-- ==================== -->
   <!-- PROPELLERS (프로펠러) -->
@@ -211,4 +188,34 @@
     <child link="imu_link"/>
     <origin xyz="0 0 ${body_height + 0.01}" rpy="0 0 0"/>
+  </joint>
+  <!-- Camera -->
+  <link name="camera_link">
+    <visual>
+      <geometry>
+        <box size="0.02 0.04 0.02"/>
+      </geometry>
+      <material name="black"/>
+    </visual>
+    <collision>
+      <geometry>
+        <box size="0.02 0.04 0.02"/>
+      </geometry>
+    </collision>
+    <inertial>
+      <mass value="0.05"/>
+      <xacro:box_inertia m="0.05" x="0.02" y="0.04" z="0.02"/>
+    </inertial>
+  </link>
+  <joint name="camera_joint" type="fixed">
+    <parent link="base_link"/>
+    <child link="camera_link"/>
+    <origin xyz="${body_length/2} 0 ${body_height/2 + 0.02}" rpy="0 0 0"/>
+  </joint>
+  <!-- Camera optical frame (ROS convention: Z forward, X right, Y down) -->
+  <link name="camera_optical_frame"/>
+  <joint name="camera_optical_joint" type="fixed">
+    <parent link="camera_link"/>
+    <child link="camera_optical_frame"/>
+    <origin xyz="0 0 0" rpy="${-pi/2} 0 ${-pi/2}"/>
   </joint>
   <!-- LiDAR (옵션) -->
@@ -238,9 +245,13 @@
   <!-- GAZEBO PLUGINS       -->
   <!-- ==================== -->
-  <!-- Differential Drive (지상 모드) -->
+  <!-- Skid Steer Drive (4바퀴) -->
   <gazebo>
     <plugin filename="gz-sim-diff-drive-system" name="gz::sim::systems::DiffDrive">
-      <left_joint>left_wheel_joint</left_joint>
-      <right_joint>right_wheel_joint</right_joint>
+      <!-- 왼쪽 바퀴들 -->
+      <left_joint>front_left_wheel_joint</left_joint>
+      <left_joint>rear_left_wheel_joint</left_joint>
+      <!-- 오른쪽 바퀴들 -->
+      <right_joint>front_right_wheel_joint</right_joint>
+      <right_joint>rear_right_wheel_joint</right_joint>
       <wheel_separation>${wheel_base}</wheel_separation>
       <wheel_radius>${wheel_radius}</wheel_radius>
@@ -258,6 +269,10 @@
     <plugin filename="gz-sim-joint-state-publisher-system" name="gz::sim::systems::JointStatePublisher">
       <topic>joint_states</topic>
-      <joint_name>left_wheel_joint</joint_name>
-      <joint_name>right_wheel_joint</joint_name>
+      <!-- 4바퀴 조인트 -->
+      <joint_name>front_left_wheel_joint</joint_name>
+      <joint_name>front_right_wheel_joint</joint_name>
+      <joint_name>rear_left_wheel_joint</joint_name>
+      <joint_name>rear_right_wheel_joint</joint_name>
+      <!-- 프로펠러 조인트 -->
       <joint_name>front_left_propeller_joint</joint_name>
       <joint_name>front_right_propeller_joint</joint_name>
@@ -299,3 +314,23 @@
     </sensor>
   </gazebo>
+  <!-- Camera Sensor -->
+  <gazebo reference="camera_link">
+    <sensor name="camera" type="camera">
+      <topic>camera/image_raw</topic>
+      <update_rate>30</update_rate>
+      <gz_frame_id>camera_optical_frame</gz_frame_id>
+      <camera>
+        <horizontal_fov>1.3962634</horizontal_fov>
+        <image>
+          <width>640</width>
+          <height>480</height>
+          <format>R8G8B8</format>
+        </image>
+        <clip>
+          <near>0.02</near>
+          <far>100</far>
+        </clip>
+      </camera>
+    </sensor>
+  </gazebo>
 </robot>

Commit message: Add STL meshes and update URDF for robot visualization
- Add full robot STL mesh (drobot_body.stl)
- Add separate part STL files (body, legs, wheels) for future use
- Update URDF to use STL mesh with proper origin alignment
- Remove sensor visual geometries (included in STL)
- Update CLAUDE.md and README.md

Co-Authored-By: Claude Opus 4.5 <noreply@anthropic.com>

File: drobot_simulation/urdf/drobot.urdf.xacro (robot description, xacro)
@@ -49,14 +49,7 @@
              izz="${m*r*r/2}"/>
   </xacro:macro>
-  <!-- 바퀴 매크로 (4바퀴 지원) -->
+  <!-- 바퀴 매크로 (visual 제거 - 통째 STL에 포함) -->
   <xacro:macro name="wheel" params="prefix x_offset y_offset">
     <link name="${prefix}_wheel">
-      <visual>
-        <geometry>
-          <cylinder radius="${wheel_radius}" length="${wheel_width}"/>
-        </geometry>
-        <origin xyz="0 0 0" rpy="${pi/2} 0 0"/>
-        <material name="black"/>
-      </visual>
       <collision>
         <geometry>
@@ -126,12 +119,11 @@
   <link name="base_footprint"/>
   <link name="base_link">
-    <visual>
-      <geometry>
-        <!-- STL 파일로 교체하려면 아래 주석 해제 -->
-        <!-- <mesh filename="package://drobot_simulation/meshes/drone_body.stl" scale="0.001 0.001 0.001"/> -->
-        <box size="${body_length} ${body_width} ${body_height}"/>
-      </geometry>
-      <origin xyz="0 0 ${body_height/2}" rpy="0 0 0"/>
-      <material name="blue"/>
+    <!-- 통째 STL -->
+    <visual name="body_mesh">
+      <geometry>
+        <mesh filename="package://drobot_simulation/meshes/drobot_body.stl" scale="0.001 0.001 0.001"/>
+      </geometry>
+      <origin xyz="0 0 -0.05" rpy="1.5708 0 0"/>
+      <material name="orange"/>
     </visual>
     <collision>
@@ -165,22 +157,8 @@
   <xacro:wheel prefix="rear_right"  x_offset="${-wheel_separation_length/2}" y_offset="${-wheel_base/2}"/>
   <!-- ==================== -->
-  <!-- PROPELLERS (프로펠러) -->
-  <!-- ==================== -->
-  <!-- 쿼드콥터 배치: X 형태 -->
-  <xacro:propeller prefix="front_left"  x_offset="${arm_length * 0.707}"  y_offset="${arm_length * 0.707}"  rotation_dir="cw"/>
-  <xacro:propeller prefix="front_right" x_offset="${arm_length * 0.707}"  y_offset="${-arm_length * 0.707}" rotation_dir="ccw"/>
-  <xacro:propeller prefix="rear_left"   x_offset="${-arm_length * 0.707}" y_offset="${arm_length * 0.707}"  rotation_dir="ccw"/>
-  <xacro:propeller prefix="rear_right"  x_offset="${-arm_length * 0.707}" y_offset="${-arm_length * 0.707}" rotation_dir="cw"/>
-  <!-- ==================== -->
   <!-- SENSORS              -->
   <!-- ==================== -->
-  <!-- IMU -->
+  <!-- IMU (visual 제거 - STL에 포함) -->
   <link name="imu_link">
-    <visual>
-      <geometry>
-        <box size="0.02 0.02 0.01"/>
-      </geometry>
-      <material name="orange"/>
-    </visual>
   </link>
   <joint name="imu_joint" type="fixed">
@@ -189,12 +167,6 @@
     <origin xyz="0 0 ${body_height + 0.01}" rpy="0 0 0"/>
   </joint>
-  <!-- Camera -->
+  <!-- Camera (visual 제거 - STL에 포함) -->
   <link name="camera_link">
-    <visual>
-      <geometry>
-        <box size="0.02 0.04 0.02"/>
-      </geometry>
-      <material name="black"/>
-    </visual>
     <collision>
       <geometry>
@@ -219,12 +191,6 @@
     <origin xyz="0 0 0" rpy="${-pi/2} 0 ${-pi/2}"/>
   </joint>
-  <!-- LiDAR (옵션) -->
+  <!-- LiDAR (visual 제거 - STL에 포함) -->
   <link name="lidar_link">
-    <visual>
-      <geometry>
-        <cylinder radius="0.03" length="0.04"/>
-      </geometry>
-      <material name="black"/>
-    </visual>
     <collision>
       <geometry>
@@ -276,9 +242,4 @@
       <joint_name>rear_left_wheel_joint</joint_name>
       <joint_name>rear_right_wheel_joint</joint_name>
-      <!-- 프로펠러 조인트 -->
-      <joint_name>front_left_propeller_joint</joint_name>
-      <joint_name>front_right_propeller_joint</joint_name>
-      <joint_name>rear_left_propeller_joint</joint_name>
-      <joint_name>rear_right_propeller_joint</joint_name>
     </plugin>
   </gazebo>

Commit message: Improve auto exploration and add project roadmap
- Add project roadmap (Phase 1: Ground, Phase 2: Drone, Phase 3: Hybrid)
- Update README with tech stack comparison and PX4 setup guide
- Fix LiDAR alignment issue (adjust lidar_joint position)
- Tune auto_explorer parameters for better navigation:
  - Increase collision distance threshold (0.38m → 0.50m)
  - Relax oscillation detection (threshold 5 → 8)
  - Increase no-progress timeout (6s → 10s)
- Reduce robot_radius for costmap (0.05m → 0.01m)
- Update SLAM/EKF parameters for better rotation tracking

Co-Authored-By: Claude Opus 4.5 <noreply@anthropic.com>

File: drobot_simulation/urdf/drobot.urdf.xacro (robot description, xacro)
@@ -124,5 +124,6 @@
         <mesh filename="package://drobot_simulation/meshes/drobot_body.stl" scale="0.001 0.001 0.001"/>
       </geometry>
-      <origin xyz="0 0 -0.05" rpy="1.5708 0 0"/>
+      <!-- STL 원점 보정: 로봇 중심으로 이동 -->
+      <origin xyz="-0.18 0.2 -0.05" rpy="1.5708 0 0"/>
       <material name="orange"/>
     </visual>
@@ -206,5 +207,6 @@
     <parent link="base_link"/>
     <child link="lidar_link"/>
-    <origin xyz="0 0 ${body_height + 0.05}" rpy="0 0 0"/>
+    <!-- LiDAR 위치 보정: 스캔이 앞+오른쪽으로 밀려서 앞+오른쪽으로 이동 -->
+    <origin xyz="0.05 -0.05 ${body_height + 0.05}" rpy="0 0 0"/>
   </joint>
   <!-- ==================== -->
@@ -269,5 +271,5 @@
         </scan>
         <range>
-          <min>0.1</min>
+          <min>0.35</min>
           <max>12.0</max>
           <resolution>0.01</resolution>
