Commit message: feat: drobot_desc 4WD diff-drive 주행 성공
- drobot_desc 패키지 추가 (SW2URDF 기반 새 URDF)
- 왼쪽 바퀴 축 반전 (0,0,-1) — 좌우 회전 방향 일치
- 바퀴 mesh 중심을 회전축에 정렬 (visual/collision origin 보정)
- joint origin 보상으로 바퀴 위치 유지
- DiffDrive 플러그인에 4바퀴 등록 (앞+뒤)
- arm joint를 fixed로 변경 (주행 테스트용)
- GZ_SIM_RESOURCE_PATH 설정으로 Gazebo mesh 로딩 해결
- 기존 drobot_description에 COLCON_IGNORE 추가

Co-Authored-By: Claude Opus 4.6 <noreply@anthropic.com>

File: drobot_description/urdf/drobot.urdf.xacro (robot description, xacro)
@@ -1,301 +1,341 @@
 <?xml version="1.0"?>
-<robot name="drobot" xmlns:xacro="http://www.ros.org/wiki/xacro">
-  <!-- ==================== -->
-  <!-- PARAMETERS           -->
-  <!-- ==================== -->
-  <!-- 로봇 크기 (미터 단위) - Onshape에서 측정 후 수정하세요 -->
-  <xacro:property name="body_length" value="0.30"/>
-  <xacro:property name="body_width" value="0.20"/>
-  <xacro:property name="body_height" value="0.10"/>
-  <xacro:property name="body_mass" value="1.5"/>
-  <!-- 바퀴 파라미터 -->
-  <xacro:property name="wheel_radius" value="0.05"/>
-  <xacro:property name="wheel_width" value="0.04"/>
-  <xacro:property name="wheel_mass" value="0.2"/>
-  <xacro:property name="wheel_base" value="0.24"/>  <!-- 좌우 바퀴 간 거리 -->
-  <xacro:property name="wheel_separation_length" value="0.20"/>  <!-- 앞뒤 바퀴 간 거리 -->
-  <!-- 프로펠러 파라미터 -->
-  <xacro:property name="prop_radius" value="0.08"/>
-  <xacro:property name="prop_height" value="0.01"/>
-  <xacro:property name="prop_mass" value="0.05"/>
-  <xacro:property name="arm_length" value="0.15"/>  <!-- 중심에서 프로펠러까지 -->
-  <!-- ==================== -->
-  <!-- MATERIALS            -->
-  <!-- ==================== -->
-  <material name="blue">
-    <color rgba="0.2 0.4 0.8 1.0"/>
-  </material>
-  <material name="black">
-    <color rgba="0.1 0.1 0.1 1.0"/>
-  </material>
-  <material name="orange">
-    <color rgba="1.0 0.5 0.0 1.0"/>
-  </material>
-  <material name="gray">
-    <color rgba="0.5 0.5 0.5 1.0"/>
-  </material>
-  <!-- ==================== -->
-  <!-- MACROS               -->
-  <!-- ==================== -->
-  <!-- Inertia 계산 매크로 -->
-  <xacro:macro name="box_inertia" params="m x y z">
-    <inertia ixx="${m*(y*y+z*z)/12}" ixy="0" ixz="0"
-             iyy="${m*(x*x+z*z)/12}" iyz="0"
-             izz="${m*(x*x+y*y)/12}"/>
-  </xacro:macro>
-  <xacro:macro name="cylinder_inertia" params="m r h">
-    <inertia ixx="${m*(3*r*r+h*h)/12}" ixy="0" ixz="0"
-             iyy="${m*(3*r*r+h*h)/12}" iyz="0"
-             izz="${m*r*r/2}"/>
-  </xacro:macro>
-  <!-- 바퀴 매크로 (visual 제거 - 통째 STL에 포함) -->
-  <xacro:macro name="wheel" params="prefix x_offset y_offset">
-    <link name="${prefix}_wheel">
-      <collision>
-        <geometry>
-          <cylinder radius="${wheel_radius}" length="${wheel_width}"/>
-        </geometry>
-        <origin xyz="0 0 0" rpy="${pi/2} 0 0"/>
-      </collision>
-      <inertial>
-        <mass value="${wheel_mass}"/>
-        <origin xyz="0 0 0" rpy="${pi/2} 0 0"/>
-        <xacro:cylinder_inertia m="${wheel_mass}" r="${wheel_radius}" h="${wheel_width}"/>
-      </inertial>
-    </link>
-    <joint name="${prefix}_wheel_joint" type="continuous">
-      <parent link="base_link"/>
-      <child link="${prefix}_wheel"/>
-      <origin xyz="${x_offset} ${y_offset} 0" rpy="0 0 0"/>
-      <axis xyz="0 1 0"/>
-      <dynamics damping="0.1" friction="0.1"/>
-    </joint>
-    <!-- Gazebo 바퀴 마찰 설정 -->
-    <gazebo reference="${prefix}_wheel">
-      <mu1>1.0</mu1>
-      <mu2>1.0</mu2>
-      <kp>1000000.0</kp>
-      <kd>100.0</kd>
-      <material>Gazebo/DarkGrey</material>
-    </gazebo>
-  </xacro:macro>
-  <!-- 프로펠러 매크로 -->
-  <xacro:macro name="propeller" params="prefix x_offset y_offset rotation_dir">
-    <link name="${prefix}_propeller">
-      <visual>
-        <geometry>
-          <!-- STL 파일로 교체하려면 아래 주석 해제 -->
-          <!-- <mesh filename="package://drobot_description/meshes/propeller.stl" scale="0.001 0.001 0.001"/> -->
-          <cylinder radius="${prop_radius}" length="${prop_height}"/>
-        </geometry>
-        <origin xyz="0 0 0" rpy="0 0 0"/>
-        <material name="gray"/>
-      </visual>
-      <collision>
-        <geometry>
-          <cylinder radius="${prop_radius}" length="${prop_height}"/>
-        </geometry>
-        <origin xyz="0 0 0" rpy="0 0 0"/>
-      </collision>
-      <inertial>
-        <mass value="${prop_mass}"/>
-        <xacro:cylinder_inertia m="${prop_mass}" r="${prop_radius}" h="${prop_height}"/>
-      </inertial>
-    </link>
-    <joint name="${prefix}_propeller_joint" type="continuous">
-      <parent link="base_link"/>
-      <child link="${prefix}_propeller"/>
-      <origin xyz="${x_offset} ${y_offset} ${body_height/2 + 0.02}" rpy="0 0 0"/>
-      <axis xyz="0 0 1"/>
-      <dynamics damping="0.001"/>
-    </joint>
-    <gazebo reference="${prefix}_propeller">
-      <material>Gazebo/Grey</material>
-    </gazebo>
-  </xacro:macro>
-  <!-- ==================== -->
-  <!-- BASE LINK (본체)     -->
-  <!-- ==================== -->
+<robot xmlns:xacro="http://ros.org/wiki/xacro" name="drobot">
+  <!-- ============================================================
+       DROBOT - SW2URDF Export → ROS2 변환
+       좌표/mesh는 SW2URDF 자동생성값 그대로 사용
+       Joint type, mimic, gazebo 플러그인 수동 추가
+       ============================================================ -->
+  <xacro:include filename="$(find drobot_description)/urdf/gazebo.xacro"/>
+  <xacro:arg name="use_sim" default="true"/>
+  <xacro:arg name="use_ros2_control" default="true"/>
+  <!-- ==================== MATERIALS ==================== -->
+  <material name="base_color"><color rgba="0.81 0.86 0.90 1"/></material>
+  <material name="arm_color"><color rgba="0.87 0.32 0.16 1"/></material>
+  <material name="frame_color"><color rgba="0.30 0.30 0.30 1"/></material>
+  <material name="wheel_color"><color rgba="0.65 0.65 0.65 1"/></material>
+  <!-- ==================== BASE ==================== -->
   <link name="base_footprint"/>
-  <link name="base_link">
-    <!-- 통째 STL -->
-    <visual name="body_mesh">
-      <geometry>
-        <mesh filename="package://drobot_description/meshes/drobot_body.stl" scale="0.001 0.001 0.001"/>
-      </geometry>
-      <!-- STL 원점 보정: 로봇 중심으로 이동 -->
-      <origin xyz="-0.18 0.2 -0.05" rpy="1.5708 0 0"/>
-      <material name="orange"/>
-    </visual>
-    <collision>
-      <geometry>
-        <box size="${body_length} ${body_width} ${body_height}"/>
-      </geometry>
-      <origin xyz="0 0 ${body_height/2}" rpy="0 0 0"/>
-    </collision>
-    <inertial>
-      <mass value="${body_mass}"/>
-      <origin xyz="0 0 ${body_height/2}" rpy="0 0 0"/>
-      <xacro:box_inertia m="${body_mass}" x="${body_length}" y="${body_width}" z="${body_height}"/>
-    </inertial>
-  </link>
   <joint name="base_footprint_joint" type="fixed">
     <parent link="base_footprint"/>
     <child link="base_link"/>
-    <origin xyz="0 0 ${wheel_radius}" rpy="0 0 0"/>
-  </joint>
-  <gazebo reference="base_link">
-    <material>Gazebo/Blue</material>
-  </gazebo>
-  <!-- ==================== -->
-  <!-- WHEELS (4바퀴 스키드 스티어) -->
-  <!-- ==================== -->
-  <!-- 앞바퀴 -->
-  <xacro:wheel prefix="front_left"  x_offset="${wheel_separation_length/2}"  y_offset="${wheel_base/2}"/>
-  <xacro:wheel prefix="front_right" x_offset="${wheel_separation_length/2}"  y_offset="${-wheel_base/2}"/>
-  <!-- 뒷바퀴 -->
-  <xacro:wheel prefix="rear_left"   x_offset="${-wheel_separation_length/2}" y_offset="${wheel_base/2}"/>
-  <xacro:wheel prefix="rear_right"  x_offset="${-wheel_separation_length/2}" y_offset="${-wheel_base/2}"/>
-  <!-- ==================== -->
-  <!-- SENSORS              -->
-  <!-- ==================== -->
-  <!-- IMU (visual 제거 - STL에 포함) -->
-  <link name="imu_link">
-  </link>
-  <joint name="imu_joint" type="fixed">
+    <origin xyz="0 0 0" rpy="0 0 0"/>
+  </joint>
+  <link name="base_link">
+    <inertial>
+      <origin xyz="-0.00239 -0.00675 0.19657" rpy="0 0 0"/>
+      <mass value="0.89777"/>
+      <inertia ixx="0.000894" ixy="-3.15e-05" ixz="7.38e-08"
+               iyy="0.001444" iyz="-7.35e-07" izz="0.001732"/>
+    </inertial>
+    <visual>
+      <origin xyz="0 0 0" rpy="0 0 0"/>
+      <geometry>
+        <mesh filename="package://drobot_description/meshes/base_link.STL"/>
+      </geometry>
+      <material name="base_color"/>
+    </visual>
+    <collision>
+      <origin xyz="0 0 0" rpy="0 0 0"/>
+      <geometry>
+        <mesh filename="package://drobot_description/meshes/base_link.STL"/>
+      </geometry>
+    </collision>
+  </link>
+  <!-- ==================== LEFT FRONT ARM ==================== -->
+  <link name="left_front_arm">
+    <inertial>
+      <origin xyz="-0.001 -0.21577 0.24030" rpy="0 0 0"/>
+      <mass value="0.05"/>
+      <inertia ixx="0.0001" ixy="0" ixz="0"
+               iyy="0.0001" iyz="0" izz="0.0001"/>
+    </inertial>
+    <visual>
+      <origin xyz="0 0 0" rpy="0 0 0"/>
+      <geometry>
+        <mesh filename="package://drobot_description/meshes/left_front_arm.STL"/>
+      </geometry>
+      <material name="arm_color"/>
+    </visual>
+    <collision>
+      <origin xyz="0 0 0" rpy="0 0 0"/>
+      <geometry>
+        <mesh filename="package://drobot_description/meshes/left_front_arm.STL"/>
+      </geometry>
+    </collision>
+  </link>
+  <joint name="rev_lf_arm" type="revolute">
+    <origin xyz="0.001 -0.22031 0.23615" rpy="-3.1225 0 0"/>
     <parent link="base_link"/>
-    <child link="imu_link"/>
-    <origin xyz="0 0 ${body_height + 0.01}" rpy="0 0 0"/>
-  </joint>
-  <!-- Camera (visual 제거 - STL에 포함) -->
-  <link name="camera_link">
-    <collision>
-      <geometry>
-        <box size="0.02 0.04 0.02"/>
-      </geometry>
-    </collision>
-    <inertial>
+    <child link="left_front_arm"/>
+    <axis xyz="1 0 0"/>
+    <limit lower="0" upper="${pi/2}" effort="10" velocity="1.0"/>
+    <dynamics damping="0.5" friction="0.1"/>
+  </joint>
+  <!-- ==================== LEFT SIDE FRAME ==================== -->
+  <link name="left_side_frame">
+    <inertial>
+      <origin xyz="0.000145 0.10634 0.33395" rpy="0 0 0"/>
+      <mass value="0.27356"/>
+      <inertia ixx="0.000175" ixy="1.60e-06" ixz="-1.73e-06"
+               iyy="0.002249" iyz="-5.39e-05" izz="0.002211"/>
+    </inertial>
+    <visual>
+      <origin xyz="0 0 0" rpy="0 0 0"/>
+      <geometry>
+        <mesh filename="package://drobot_description/meshes/left_side_frame.STL"/>
+      </geometry>
+      <material name="frame_color"/>
+    </visual>
+    <collision>
+      <origin xyz="0 0 0" rpy="0 0 0"/>
+      <geometry>
+        <mesh filename="package://drobot_description/meshes/left_side_frame.STL"/>
+      </geometry>
+    </collision>
+  </link>
+  <joint name="fix_ls_frame" type="fixed">
+    <origin xyz="0.0005 -0.01671 0.0040219" rpy="-0.058822 0 0"/>
+    <parent link="left_front_arm"/>
+    <child link="left_side_frame"/>
+  </joint>
+  <!-- ==================== LEFT FRONT WHEEL ==================== -->
+  <link name="left_front_wheel">
+    <inertial>
+      <origin xyz="-0.11656 0 0.02494" rpy="0 0 0"/>
+      <mass value="0.17861"/>
+      <inertia ixx="0.000611" ixy="0" ixz="0"
+               iyy="0.000611" iyz="0" izz="0.001171"/>
+    </inertial>
+    <visual>
+      <origin xyz="0 0 0" rpy="0 0 0"/>
+      <geometry>
+        <mesh filename="package://drobot_description/meshes/left_front_wheel.STL"/>
+      </geometry>
+      <material name="wheel_color"/>
+    </visual>
+    <collision>
+      <origin xyz="0 0 0" rpy="0 0 0"/>
+      <geometry>
+        <mesh filename="package://drobot_description/meshes/left_front_wheel.STL"/>
+      </geometry>
+    </collision>
+  </link>
+  <joint name="con_lf_wheel" type="continuous">
+    <origin xyz="-0.1485 0.166 0.4581" rpy="-1.5708 -1.2933 3.1416"/>
+    <parent link="left_side_frame"/>
+    <child link="left_front_wheel"/>
+    <axis xyz="0 0 1"/>
+    <dynamics damping="0.1" friction="0.05"/>
+  </joint>
+  <!-- ==================== LEFT REAR WHEEL ==================== -->
+  <link name="left_rear_wheel">
+    <inertial>
+      <origin xyz="0.11656 0 0.02435" rpy="0 0 0"/>
+      <mass value="0.17645"/>
+      <inertia ixx="0.000608" ixy="0" ixz="0"
+               iyy="0.000608" iyz="0" izz="0.001169"/>
+    </inertial>
+    <visual>
+      <origin xyz="0 0 0" rpy="0 0 0"/>
+      <geometry>
+        <mesh filename="package://drobot_description/meshes/left_rear_wheel.STL"/>
+      </geometry>
+      <material name="wheel_color"/>
+    </visual>
+    <collision>
+      <origin xyz="0 0 0" rpy="0 0 0"/>
+      <geometry>
+        <mesh filename="package://drobot_description/meshes/left_rear_wheel.STL"/>
+      </geometry>
+    </collision>
+  </link>
+  <joint name="con_lr_wheel" type="continuous">
+    <origin xyz="0.14702 0.164 0.23349" rpy="-1.5708 -1.3064 3.1416"/>
+    <parent link="left_side_frame"/>
+    <child link="left_rear_wheel"/>
+    <axis xyz="0 0 1"/>
+    <dynamics damping="0.1" friction="0.05"/>
+  </joint>
+  <!-- ==================== LEFT REAR ARM ==================== -->
+  <link name="left_rear_arm">
+    <inertial>
+      <origin xyz="0 0 0" rpy="0 0 0"/>
       <mass value="0.05"/>
-      <xacro:box_inertia m="0.05" x="0.02" y="0.04" z="0.02"/>
-    </inertial>
-  </link>
-  <joint name="camera_joint" type="fixed">
+      <inertia ixx="0.0001" ixy="0" ixz="0"
+               iyy="0.0001" iyz="0" izz="0.0001"/>
+    </inertial>
+    <visual>
+      <origin xyz="0 0 0" rpy="0 0 0"/>
+      <geometry>
+        <mesh filename="package://drobot_description/meshes/left_rear_arm.STL"/>
+      </geometry>
+      <material name="arm_color"/>
+    </visual>
+    <collision>
+      <origin xyz="0 0 0" rpy="0 0 0"/>
+      <geometry>
+        <mesh filename="package://drobot_description/meshes/left_rear_arm.STL"/>
+      </geometry>
+    </collision>
+  </link>
+  <joint name="rev_lr_arm" type="revolute">
+    <origin xyz="0 0 0" rpy="1.5898 0 0"/>
     <parent link="base_link"/>
-    <child link="camera_link"/>
-    <origin xyz="${body_length/2} 0 ${body_height/2 + 0.02}" rpy="0 0 0"/>
-  </joint>
-  <!-- Camera optical frame (ROS convention: Z forward, X right, Y down) -->
-  <link name="camera_optical_frame"/>
-  <joint name="camera_optical_joint" type="fixed">
-    <parent link="camera_link"/>
-    <child link="camera_optical_frame"/>
-    <origin xyz="0 0 0" rpy="${-pi/2} 0 ${-pi/2}"/>
-  </joint>
-  <!-- LiDAR (visual 제거 - STL에 포함) -->
-  <link name="lidar_link">
-    <collision>
-      <geometry>
-        <cylinder radius="0.03" length="0.04"/>
-      </geometry>
-    </collision>
-    <inertial>
-      <mass value="0.1"/>
-      <xacro:cylinder_inertia m="0.1" r="0.03" h="0.04"/>
-    </inertial>
-  </link>
-  <joint name="lidar_joint" type="fixed">
+    <child link="left_rear_arm"/>
+    <axis xyz="1 0 0"/>
+    <limit lower="0" upper="${pi/2}" effort="10" velocity="1.0"/>
+    <dynamics damping="0.5" friction="0.1"/>
+    <mimic joint="rev_lf_arm" multiplier="1" offset="0"/>
+  </joint>
+  <!-- ==================== RIGHT FRONT ARM ==================== -->
+  <link name="right_front_arm">
+    <inertial>
+      <origin xyz="-0.09053 0.04100 0.15322" rpy="0 0 0"/>
+      <mass value="0.09050"/>
+      <inertia ixx="7.55e-05" ixy="6.14e-06" ixz="-3.92e-06"
+               iyy="5.55e-05" iyz="2.21e-05" izz="5.80e-05"/>
+    </inertial>
+    <visual>
+      <origin xyz="0 0 0" rpy="0 0 0"/>
+      <geometry>
+        <mesh filename="package://drobot_description/meshes/right_front_arm.STL"/>
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
Commit message: Fix navigation odom/wheel issues, add hospital world models, replace yolo with perception
- Fix inverted odometry: replace DiffDrive odom with OdometryPublisher (model pose based)
- Fix backward motion: swap all wheel axis signs in URDF
- Simplify EKF: use only odom + IMU vyaw (remove acceleration conflict)
- Add 98 3D models for hospital_original world (aws_robomaker + fuel_models)
- Fix hospital_original.world physics tag (add type="ode")
- Add hospital spawn position (0, 1.5) to spawn_positions.yaml
- Replace drobot_yolo with perception package
- Update README with current setup instructions

Co-Authored-By: Claude Opus 4.6 <noreply@anthropic.com>

File: drobot_description/urdf/drobot.urdf.xacro (robot description, xacro)
@@ -111,10 +111,9 @@
     </collision>
   </link>
-  <!-- FIX: axis flipped to 0,0,-1 so left wheels match right wheels in base_link frame -->
   <joint name="con_lf_wheel" type="continuous">
     <origin xyz="-0.11657 0.14106 0.34600" rpy="-1.5708 -1.2933 3.1416"/>
     <parent link="left_side_frame"/>
     <child link="left_front_wheel"/>
-    <axis xyz="0 0 -1"/>
+    <axis xyz="0 0 1"/>
     <dynamics damping="0.1" friction="0.05"/>
   </joint>
@@ -141,10 +140,9 @@
     </collision>
   </link>
-  <!-- FIX: axis flipped to 0,0,-1 so left wheels match right wheels in base_link frame -->
   <joint name="con_lr_wheel" type="continuous">
     <origin xyz="0.11656 0.13965 0.34600" rpy="-1.5708 -1.3064 3.1416"/>
     <parent link="left_side_frame"/>
     <child link="left_rear_wheel"/>
-    <axis xyz="0 0 -1"/>
+    <axis xyz="0 0 1"/>
     <dynamics damping="0.1" friction="0.05"/>
   </joint>
@@ -245,5 +243,5 @@
     <parent link="right_side_frame"/>
     <child link="right_front_wheel"/>
-    <axis xyz="0 0 1"/>
+    <axis xyz="0 0 -1"/>
     <dynamics damping="0.1" friction="0.05"/>
   </joint>
@@ -275,5 +273,5 @@
     <parent link="right_side_frame"/>
     <child link="right_rear_wheel"/>
-    <axis xyz="0 0 1"/>
+    <axis xyz="0 0 -1"/>
     <dynamics damping="0.1" friction="0.05"/>
   </joint>

File: drobot_description/urdf/gazebo.xacro (robot description, xacro)
@@ -12,5 +12,5 @@
     </plugin>
   </gazebo>
-  <!-- Diff Drive -->
+  <!-- Diff Drive (cmd_vel only, odom disabled — wheel axes are mixed ±Z) -->
   <gazebo>
     <plugin filename="gz-sim-diff-drive-system"
@@ -23,7 +23,14 @@
       <wheel_radius>0.112</wheel_radius>
       <topic>/cmd_vel</topic>
+    </plugin>
+  </gazebo>
+  <!-- Odometry from model pose (avoids wheel axis sign issue) -->
+  <gazebo>
+    <plugin filename="gz-sim-odometry-publisher-system"
+            name="gz::sim::systems::OdometryPublisher">
+      <odom_publish_frequency>50</odom_publish_frequency>
+      <odom_frame>odom</odom_frame>
+      <robot_base_frame>base_footprint</robot_base_frame>
       <odom_topic>/odom</odom_topic>
-      <frame_id>odom</frame_id>
-      <child_frame_id>base_footprint</child_frame_id>
     </plugin>
   </gazebo>
