Commit message: Add camera link and sensor for Gazebo perception pipeline
- Add camera_link and camera_joint to URDF (front of robot, xyz 0 -0.22 0.05)
- Add camera sensor plugin to gazebo.xacro (640x480, 15Hz, /camera/image_raw)
- Fix wheel axis signs: left wheels 0,0,1→0,0,-1, right wheels 0,0,-1→0,0,1

Co-Authored-By: Claude Opus 4.6 <noreply@anthropic.com>

File: src/drobot_description/urdf/drobot.urdf.xacro (robot description, xacro)
@@ -2,6 +2,4 @@
 <robot xmlns:xacro="http://ros.org/wiki/xacro" name="drobot">
   <!-- ============================================================
-       DROBOT - SW2URDF FINAL Export → ROS2 변환
-       좌표/mesh: SW2URDF 자동생성값 그대로
        수동 수정: mass=0 fix, axis fix, limit/dynamics, mimic, gazebo
        ============================================================ -->
@@ -111,9 +109,10 @@
     </collision>
   </link>
+  <!-- FIX: axis flipped to 0,0,-1 so left wheels match right wheels in base_link frame -->
   <joint name="con_lf_wheel" type="continuous">
     <origin xyz="-0.11657 0.14106 0.34600" rpy="-1.5708 -1.2933 3.1416"/>
     <parent link="left_side_frame"/>
     <child link="left_front_wheel"/>
-    <axis xyz="0 0 1"/>
+    <axis xyz="0 0 -1"/>
     <dynamics damping="0.1" friction="0.05"/>
   </joint>
@@ -140,9 +139,10 @@
     </collision>
   </link>
+  <!-- FIX: axis flipped to 0,0,-1 so left wheels match right wheels in base_link frame -->
   <joint name="con_lr_wheel" type="continuous">
     <origin xyz="0.11656 0.13965 0.34600" rpy="-1.5708 -1.3064 3.1416"/>
     <parent link="left_side_frame"/>
     <child link="left_rear_wheel"/>
-    <axis xyz="0 0 1"/>
+    <axis xyz="0 0 -1"/>
     <dynamics damping="0.1" friction="0.05"/>
   </joint>
@@ -243,5 +243,5 @@
     <parent link="right_side_frame"/>
     <child link="right_front_wheel"/>
-    <axis xyz="0 0 -1"/>
+    <axis xyz="0 0 1"/>
     <dynamics damping="0.1" friction="0.05"/>
   </joint>
@@ -273,5 +273,5 @@
     <parent link="right_side_frame"/>
     <child link="right_rear_wheel"/>
-    <axis xyz="0 0 -1"/>
+    <axis xyz="0 0 1"/>
     <dynamics damping="0.1" friction="0.05"/>
   </joint>
@@ -333,4 +333,24 @@
     <child link="imu_link"/>
     <origin xyz="0 -0.19 0.02" rpy="0 0 0"/>
+  </joint>
+  <!-- ==================== CAMERA ==================== -->
+  <link name="camera_link">
+    <inertial>
+      <origin xyz="0 0 0" rpy="0 0 0"/>
+      <mass value="0.01"/>
+      <inertia ixx="1e-06" ixy="0" ixz="0" iyy="1e-06" iyz="0" izz="1e-06"/>
+    </inertial>
+    <visual>
+      <origin xyz="0 0 0" rpy="0 0 0"/>
+      <geometry>
+        <box size="0.02 0.04 0.02"/>
+      </geometry>
+      <material name="frame_color"/>
+    </visual>
+  </link>
+  <joint name="camera_joint" type="fixed">
+    <parent link="base_link"/>
+    <child link="camera_link"/>
+    <origin xyz="0 -0.22 0.05" rpy="0 0 0"/>
   </joint>
   <!-- ==================== ROS2 CONTROL ==================== -->

File: src/drobot_description/urdf/gazebo.xacro (robot description, xacro)
@@ -123,4 +123,26 @@
     </sensor>
   </gazebo>
+  <!-- ========== CAMERA ========== -->
+  <gazebo reference="camera_link">
+    <sensor name="camera" type="camera">
+      <topic>/camera/image_raw</topic>
+      <gz_frame_id>camera_link</gz_frame_id>
+      <update_rate>15</update_rate>
+      <always_on>true</always_on>
+      <visualize>false</visualize>
+      <camera>
+        <horizontal_fov>1.047</horizontal_fov>
+        <image>
+          <width>640</width>
+          <height>480</height>
+          <format>R8G8B8</format>
+        </image>
+        <clip>
+          <near>0.1</near>
+          <far>100</far>
+        </clip>
+      </camera>
+    </sensor>
+  </gazebo>
   <!-- Wheel Friction -->
   <gazebo reference="left_front_wheel">

Commit message: Fix camera orientation and position to face robot forward (-Y)
- Move camera further forward (Y=-0.40) and higher (Z=0.15) to clear robot body
- Set yaw to -180° so camera faces -Y direction (robot front)

Co-Authored-By: Claude Opus 4.6 <noreply@anthropic.com>

File: src/drobot_description/urdf/drobot.urdf.xacro (robot description, xacro)
@@ -352,5 +352,5 @@
     <parent link="base_link"/>
     <child link="camera_link"/>
-    <origin xyz="0 -0.22 0.05" rpy="0 0 0"/>
+    <origin xyz="0 -0.40 0.15" rpy="0 0 -3.14159"/>
   </joint>
   <!-- ==================== ROS2 CONTROL ==================== -->
