Commit message: Fix wheel rotation asymmetry and tune navigation parameters
- Wheel collision: cylinder → STL mesh (fixes left/right rotation asymmetry)
- Arm joint angles: exact π, π/2 values, mass/inertia equalized
- Gazebo: mu2=0.15, wheel_separation=0.35
- Nav2: RotationShimController for heading alignment before path following
- Nav2: DWB forward-only (min_vel_x=0.0), oscillation critic added
- Nav2: reduced footprint/inflation for narrow passage navigation
- Nav2: global replan rate 0.5→1.0Hz, costmap update 2→5Hz
- Safety: COLLISION_STOP_DIST 0.40→0.25m

Co-Authored-By: Claude Opus 4.6 <noreply@anthropic.com>

File: src/drobot_description/urdf/drobot.urdf.xacro (robot description, xacro)
@@ -2,5 +2,13 @@
 <robot xmlns:xacro="http://ros.org/wiki/xacro" name="drobot">
   <!-- ============================================================
-       수동 수정: mass=0 fix, axis fix, limit/dynamics, mimic, gazebo
+       Source: drobotttt_urdf (SolidWorks SW2URDF export, Feb 2026)
+       Modifications:
+       - ROS1 catkin -> ROS2 ament, .urdf -> .urdf.xacro
+       - mesh paths: package://drobot_description/meshes/
+       - base_footprint added (z=0.25 offset)
+       - left_rear_arm mass=0 -> 0.05 + min inertia
+       - arm dynamics: damping=5.0 friction=1.0
+       - wheel dynamics: damping=0.1 friction=0.05
+       - left wheel axis flipped (0,-1,0) -> (0,1,0) for DiffDrive
        ============================================================ -->
   <xacro:include filename="$(find drobot_description)/urdf/gazebo.xacro"/>
@@ -12,4 +20,5 @@
   <material name="frame_color"><color rgba="0.30 0.30 0.30 1"/></material>
   <material name="wheel_color"><color rgba="0.65 0.65 0.65 1"/></material>
+  <material name="sensor_color"><color rgba="0.79 0.82 0.93 1"/></material>
   <!-- ==================== BASE ==================== -->
   <link name="base_footprint"/>
@@ -17,71 +26,128 @@
     <parent link="base_footprint"/>
     <child link="base_link"/>
-    <!-- z offset: base_footprint(지면)에서 base_link까지 높이 -->
     <origin xyz="0 0 0.25" rpy="0 0 0"/>
   </joint>
   <link name="base_link">
     <inertial>
-      <origin xyz="-0.0023939 -0.19657 -0.0067497" rpy="0 0 0"/>
-      <mass value="0.89777"/>
-      <inertia ixx="0.00089357" ixy="-7.3792e-08" ixz="-3.1542e-05"
-               iyy="0.0017315" iyz="7.3533e-07" izz="0.0014439"/>
-    </inertial>
-    <visual>
-      <origin xyz="0 0 0" rpy="0 0 0"/>
-      <geometry>
-        <mesh filename="package://drobot_description/meshes/base_link.STL"/>
-      </geometry>
+      <origin xyz="0.00458103694773914 -0.00104664211572963 0.221167547284754" rpy="0 0 0"/>
+      <mass value="0.832637440945029"/>
+      <inertia ixx="0.000773069077682801" ixy="-7.38474804169069E-08" ixz="3.15446327066613E-05"
+               iyy="0.00170450440360595" iyz="9.65699121565219E-07" izz="0.00134874358561967"/>
+    </inertial>
+    <visual>
+      <origin xyz="0 0 0" rpy="0 0 0"/>
+      <geometry><mesh filename="package://drobot_description/meshes/base_link.STL"/></geometry>
       <material name="base_color"/>
     </visual>
     <collision>
       <origin xyz="0 0 0" rpy="0 0 0"/>
-      <geometry>
-        <mesh filename="package://drobot_description/meshes/base_link.STL"/>
-      </geometry>
-    </collision>
-  </link>
+      <geometry><mesh filename="package://drobot_description/meshes/base_link.STL"/></geometry>
+    </collision>
+  </link>
+  <!-- ==================== LIDAR ==================== -->
+  <link name="lidar">
+    <inertial>
+      <origin xyz="-0.0215847721606996 0.00397566854868606 -0.00218033584701988" rpy="0 0 0"/>
+      <mass value="0.00105539669078503"/>
+      <inertia ixx="1.6596115838381E-08" ixy="4.5351666504703E-24" ixz="-8.45778550488722E-25"
+               iyy="1.98921505758854E-08" iyz="2.17400907909987E-25" izz="2.93717011285355E-08"/>
+    </inertial>
+    <visual>
+      <origin xyz="0 0 0" rpy="0 0 0"/>
+      <geometry><mesh filename="package://drobot_description/meshes/lidar.STL"/></geometry>
+      <material name="sensor_color"/>
+    </visual>
+    <collision>
+      <origin xyz="0 0 0" rpy="0 0 0"/>
+      <geometry><mesh filename="package://drobot_description/meshes/lidar.STL"/></geometry>
+    </collision>
+  </link>
+  <joint name="lidar_joint" type="fixed">
+    <origin xyz="0.010101 -0.027788 0.30154" rpy="3.1416 0 3.1416"/>
+    <parent link="base_link"/>
+    <child link="lidar"/>
+  </joint>
+  <!-- ==================== CAMERA ==================== -->
+  <link name="camera">
+    <inertial>
+      <origin xyz="-0.0215847721606996 0.00397566854868603 -0.00218033584701988" rpy="3.1416 0 3.1416"/>
+      <mass value="0.00105539669078502"/>
+      <inertia ixx="1.65961158383809E-08" ixy="-6.9134081160347E-24" ixz="-1.3026067311437E-23"
+               iyy="1.98921505758854E-08" iyz="1.59079600624928E-24" izz="2.93717011285354E-08"/>
+    </inertial>
+    <visual>
+      <origin xyz="0 0 0" rpy="3.1416 0 3.1416"/>
+      <geometry><mesh filename="package://drobot_description/meshes/camera.STL"/></geometry>
+      <material name="sensor_color"/>
+    </visual>
+    <collision>
+      <origin xyz="0 0 0" rpy="3.1416 0 3.1416"/>
+      <geometry><mesh filename="package://drobot_description/meshes/camera.STL"/></geometry>
+    </collision>
+  </link>
+  <joint name="camera_joint" type="fixed">
+    <origin xyz="0.010101 -0.027788 0.36" rpy="0 0 0"/>
+    <parent link="base_link"/>
+    <child link="camera"/>
+  </joint>
+  <!-- ==================== IMU (virtual, no mesh) ==================== -->
+  <link name="imu_link">
+    <inertial>
+      <origin xyz="0 0 0" rpy="0 0 0"/>
+      <mass value="0.01"/>
+      <inertia ixx="1e-06" ixy="0" ixz="0" iyy="1e-06" iyz="0" izz="1e-06"/>
+    </inertial>
+  </link>
+  <joint name="imu_joint" type="fixed">
+    <parent link="base_link"/>
+    <child link="imu_link"/>
+    <origin xyz="0 0 0.01" rpy="0 0 0"/>
+  </joint>
   <!-- ==================== LEFT FRONT ARM ==================== -->
-  <!-- FIX: mass was 0, set to 0.05 with minimal inertia -->
   <link name="left_front_arm">
     <inertial>
-      <origin xyz="-0.001 -0.21577 0.2403" rpy="0 0 0"/>
-      <mass value="0.05"/>
-      <inertia ixx="1e-04" ixy="0" ixz="0"
-               iyy="1e-04" iyz="0" izz="1e-04"/>
-    </inertial>
-    <visual>
-      <origin xyz="0 0 0" rpy="0 0 0"/>
-      <geometry>
-        <mesh filename="package://drobot_description/meshes/left_front_arm.STL"/>
-      </geometry>
+      <origin xyz="0.018998 -0.000534 0.112534" rpy="0 0 0"/>
+      <mass value="0.123064431731573"/>
+      <inertia ixx="0.000135741612972814" ixy="6.13644622591408E-06" ixz="-3.91949328277525E-06"
+               iyy="6.76036048729945E-05" iyz="4.48906032629936E-05" izz="0.000106939767969889"/>
+    </inertial>
+    <visual>
+      <origin xyz="0 -0.003671 -0.216881" rpy="0 0 0"/>
+      <geometry><mesh filename="package://drobot_description/meshes/left_front_arm.STL"/></geometry>
       <material name="arm_color"/>
     </visual>
-  </link>
-  <joint name="rev_lf_arm" type="revolute">
-    <origin xyz="0.001 -0.22031 0.23615" rpy="-3.1225 0 0"/>
+    <collision>
+      <origin xyz="0 -0.003671 -0.216881" rpy="0 0 0"/>
+      <geometry><mesh filename="package://drobot_description/meshes/left_front_arm.STL"/></geometry>
+    </collision>
+  </link>
+  <joint name="lf_arm_rev" type="revolute">
+    <origin xyz="0.001 0.022 0.240" rpy="3.1416 0 3.1416"/>
     <parent link="base_link"/>
     <child link="left_front_arm"/>
     <axis xyz="-1 0 0"/>
-    <limit lower="0" upper="1.5708" effort="100" velocity="2.0"/>
-    <dynamics damping="100.0" friction="1.0"/>
+    <limit lower="0" upper="1.5708" effort="100" velocity="2"/>
+    <dynamics damping="500.0" friction="50.0"/>
   </joint>
   <!-- ==================== LEFT SIDE FRAME ==================== -->
   <link name="left_side_frame">
     <inertial>
-      <origin xyz="0.00014502 0.10634 0.33395" rpy="0 0 0"/>
-      <mass value="0.27356"/>
-      <inertia ixx="0.00017455" ixy="1.6016e-06" ixz="-1.7253e-06"
-               iyy="0.0022493" iyz="-5.3889e-05" izz="0.0022114"/>
-    </inertial>
-    <visual>
-      <origin xyz="0 0 0" rpy="0 0 0"/>
-      <geometry>
-        <mesh filename="package://drobot_description/meshes/left_side_frame.STL"/>
-      </geometry>
+      <origin xyz="0.000123207540564108 0.109960226689103 0.335761073502946" rpy="0 0 0"/>
+      <mass value="0.385275324463581"/>
+      <inertia ixx="0.000226753304752499" ixy="-1.11398827218514E-05" ixz="6.22551133000347E-06"
+               iyy="0.00238329526316141" iyz="-5.33911597507339E-05" izz="0.00245899243822558"/>
+    </inertial>
+    <visual>
+      <origin xyz="0 0 0" rpy="0 0 0"/>
+      <geometry><mesh filename="package://drobot_description/meshes/left_side_frame.STL"/></geometry>
       <material name="frame_color"/>
     </visual>
-  </link>
-  <joint name="fix_ls_frame" type="fixed">
-    <origin xyz="0.0005 -0.01671 0.0040219" rpy="-0.058822 0 0"/>
+    <collision>
+      <origin xyz="0 0 0" rpy="0 0 0"/>
+      <geometry><mesh filename="package://drobot_description/meshes/left_side_frame.STL"/></geometry>
+    </collision>
+  </link>
+  <joint name="left_sf_fix" type="fixed">
+    <origin xyz="0.0005 -0.000798 -0.217469" rpy="0.010035 0 0"/>
     <parent link="left_front_arm"/>
     <child link="left_side_frame"/>
@@ -90,29 +156,29 @@
   <link name="left_front_wheel">
     <inertial>
-      <origin xyz="0 0 0" rpy="0 0 0"/>
-      <mass value="0.17861"/>
-      <inertia ixx="0.00061079" ixy="0" ixz="0"
-               iyy="0.00061079" iyz="0" izz="0.0011712"/>
-    </inertial>
-    <visual>
-      <origin xyz="0.11656 0 -0.024937" rpy="0 0 0"/>
-      <geometry>
-        <mesh filename="package://drobot_description/meshes/left_front_wheel.STL"/>
-      </geometry>
+      <origin xyz="-3.80634406216274E-08 0.0147130977298118 -4.33058131021902E-08" rpy="0 0 0"/>
+      <mass value="0.154468227846206"/>
+      <inertia ixx="0.000600972336966455" ixy="-1.7094296974559E-11" ixz="1.67775124672545E-10"
+               iyy="0.00115446036705922" iyz="-2.61109881198951E-11" izz="0.000600972175604584"/>
+    </inertial>
+    <visual>
+      <origin xyz="0 0 0" rpy="0 0 0"/>
+      <geometry><mesh filename="package://drobot_description/meshes/left_front_wheel.STL"/></geometry>
       <material name="wheel_color"/>
     </visual>
     <collision>
-      <origin xyz="0.11656 0 -0.024937" rpy="0 0 0"/>
-      <geometry>
-        <mesh filename="package://drobot_description/meshes/left_front_wheel.STL"/>
-      </geometry>
-    </collision>
-  </link>
-  <!-- FIX: axis flipped to 0,0,-1 so left wheels match right wheels in base_link frame -->
-  <joint name="con_lf_wheel" type="continuous">
-    <origin xyz="-0.11657 0.14106 0.34600" rpy="-1.5708 -1.2933 3.1416"/>
+      <origin xyz="0 0 0" rpy="0 0 0"/>
+      <geometry><mesh filename="package://drobot_description/meshes/left_front_wheel.STL"/></geometry>
+    </collision>
+  </link>
+  <!-- LEFT WHEELS: axis flipped to (0,1,0) for DiffDrive compatibility
+       Left arm rpy~(pi,0,pi) flips the Y-axis relative to base_link.
+       SW2URDF exports axis=(0,-1,0) for all wheels, but left-side Y
+       is inverted in world frame, so we flip to (0,1,0) so both sides
+       produce forward motion with positive velocity. -->
+  <joint name="lf_wheel_con" type="continuous">
+    <origin xyz="-0.11656 0.128 0.346" rpy="0 0 0"/>
     <parent link="left_side_frame"/>
     <child link="left_front_wheel"/>
-    <axis xyz="0 0 -1"/>
+    <axis xyz="0 1 0"/>
     <dynamics damping="0.1" friction="0.05"/>
   </joint>
@@ -120,98 +186,100 @@
   <link name="left_rear_wheel">
     <inertial>
-      <origin xyz="0 0 0" rpy="0 0 0"/>
-      <mass value="0.17645"/>
-      <inertia ixx="0.00060815" ixy="0" ixz="0"
-               iyy="0.00060815" iyz="0" izz="0.0011693"/>
-    </inertial>
-    <visual>
-      <origin xyz="-0.11656 0 -0.024345" rpy="0 0 0"/>
-      <geometry>
-        <mesh filename="package://drobot_description/meshes/left_rear_wheel.STL"/>
-      </geometry>
+      <origin xyz="-0.000764539518262372 0.0131052613053511 -0.000764533553625352" rpy="0 0 0"/>
+      <mass value="0.152313021640434"/>
+      <inertia ixx="0.000598326645638881" ixy="1.16817760587612E-11" ixz="1.64181067073089E-10"
+               iyy="0.00115252805512864" iyz="2.67998148070656E-11" izz="0.000598326477272364"/>
+    </inertial>
+    <visual>
+      <origin xyz="0 0 0" rpy="0 0 0"/>
+      <geometry><mesh filename="package://drobot_description/meshes/left_rear_wheel.STL"/></geometry>
       <material name="wheel_color"/>
     </visual>
     <collision>
-      <origin xyz="-0.11656 0 -0.024345" rpy="0 0 0"/>
-      <geometry>
-        <mesh filename="package://drobot_description/meshes/left_rear_wheel.STL"/>
-      </geometry>
-    </collision>
-  </link>
-  <!-- FIX: axis flipped to 0,0,-1 so left wheels match right wheels in base_link frame -->
-  <joint name="con_lr_wheel" type="continuous">
-    <origin xyz="0.11656 0.13965 0.34600" rpy="-1.5708 -1.3064 3.1416"/>
+      <origin xyz="0 0 0" rpy="0 0 0"/>
+      <geometry><mesh filename="package://drobot_description/meshes/left_rear_wheel.STL"/></geometry>
+    </collision>
+  </link>
+  <joint name="lr_wheel_con" type="continuous">
+    <origin xyz="0.11733 0.128 0.34676" rpy="0 0 0"/>
     <parent link="left_side_frame"/>
     <child link="left_rear_wheel"/>
-    <axis xyz="0 0 -1"/>
+    <axis xyz="0 1 0"/>
     <dynamics damping="0.1" friction="0.05"/>
   </joint>
   <!-- ==================== LEFT REAR ARM ==================== -->
-  <!-- FIX: mass was 0 -->
+  <!-- SW2URDF exported mass=0, inertia=0 (degenerate).
+       Fixed to mass=0.05, inertia=1e-04 for stable simulation. -->
   <link name="left_rear_arm">
     <inertial>
-      <origin xyz="0 0 0" rpy="0 0 0"/>
-      <mass value="0.05"/>
-      <inertia ixx="1e-04" ixy="0" ixz="0"
-               iyy="1e-04" iyz="0" izz="1e-04"/>
-    </inertial>
-    <visual>
-      <origin xyz="0 0 0" rpy="0 0 0"/>
-      <geometry>
-        <mesh filename="package://drobot_description/meshes/left_rear_arm.STL"/>
-      </geometry>
+      <origin xyz="-0.000999999999999908 0.00407538533818062 -0.000143536147134726" rpy="0 0 0"/>
+      <mass value="0.123064431731573"/>
+      <inertia ixx="0.000135741612972814" ixy="6.13644622591408E-06" ixz="-3.91949328277525E-06"
+               iyy="6.76036048729945E-05" iyz="4.48906032629936E-05" izz="0.000106939767969889"/>
+    </inertial>
+    <visual>
+      <origin xyz="0 0 0" rpy="0 0 0"/>
+      <geometry><mesh filename="package://drobot_description/meshes/left_rear_arm.STL"/></geometry>
       <material name="arm_color"/>
     </visual>
-  </link>
-  <joint name="rev_lr_arm" type="revolute">
-    <origin xyz="0 0 0" rpy="1.5898 0 0"/>
+    <collision>
+      <origin xyz="0 0 0" rpy="0 0 0"/>
+      <geometry><mesh filename="package://drobot_description/meshes/left_rear_arm.STL"/></geometry>
+    </collision>
+  </link>
+  <joint name="lr_arm_rev" type="revolute">
+    <origin xyz="0.001 -0.19728 0.21693" rpy="1.5708 0 3.1416"/>
     <parent link="base_link"/>
     <child link="left_rear_arm"/>
     <axis xyz="-1 0 0"/>
-    <limit lower="0" upper="1.5708" effort="100" velocity="2.0"/>
-    <dynamics damping="100.0" friction="1.0"/>
+    <limit lower="0" upper="1.5708" effort="100" velocity="2"/>
+    <dynamics damping="500.0" friction="50.0"/>
   </joint>
   <!-- ==================== RIGHT FRONT ARM ==================== -->
   <link name="right_front_arm">
     <inertial>
-      <origin xyz="-0.09053 0.041004 0.15322" rpy="0 0 0"/>
-      <mass value="0.090502"/>
-      <inertia ixx="7.5491e-05" ixy="6.1386e-06" ixz="-3.9205e-06"
-               iyy="5.5454e-05" iyz="2.2145e-05" izz="5.7986e-05"/>
-    </inertial>
-    <visual>
-      <origin xyz="0 0 0" rpy="0 0 0"/>
-      <geometry>
-        <mesh filename="package://drobot_description/meshes/right_front_arm.STL"/>
-      </geometry>
+      <origin xyz="-0.072133 0.029001 -0.051593" rpy="0 0 0"/>
+      <mass value="0.123064431731573"/>
+      <inertia ixx="0.000135741612972814" ixy="6.13644622591408E-06" ixz="-3.91949328277525E-06"
+               iyy="6.76036048729945E-05" iyz="4.48906032629936E-05" izz="0.000106939767969889"/>
+    </inertial>
+    <visual>
+      <origin xyz="0 -0.002488 -0.180993" rpy="0 0 0"/>
+      <geometry><mesh filename="package://drobot_description/meshes/right_front_arm.STL"/></geometry>
       <material name="arm_color"/>
     </visual>
-  </link>
-  <joint name="rev_rf_arm" type="revolute">
-    <origin xyz="0.001 -0.18333 -0.1565" rpy="-0.037984 0 0"/>
+    <collision>
+      <origin xyz="0 -0.002488 -0.180993" rpy="0 0 0"/>
+      <geometry><mesh filename="package://drobot_description/meshes/right_front_arm.STL"/></geometry>
+    </collision>
+  </link>
+  <joint name="rf_arm_rev" type="revolute">
+    <origin xyz="0.001 -0.023 0.245" rpy="0 0 3.1416"/>
     <parent link="base_link"/>
     <child link="right_front_arm"/>
-    <axis xyz="-1 0 0"/>
-    <limit lower="0" upper="1.5708" effort="100" velocity="2.0"/>
-    <dynamics damping="100.0" friction="1.0"/>
+    <axis xyz="1 0 0"/>
+    <limit lower="0" upper="1.5708" effort="100" velocity="2"/>
+    <dynamics damping="500.0" friction="50.0"/>
   </joint>
   <!-- ==================== RIGHT SIDE FRAME ==================== -->
   <link name="right_side_frame">
     <inertial>
-      <origin xyz="-0.0019373 0.0087805 0.060878" rpy="0 0 0"/>
-      <mass value="0.337"/>
-      <inertia ixx="0.00020711" ixy="-1.114e-05" ixz="6.2261e-06"
-               iyy="0.0023637" iyz="-5.3391e-05" izz="0.0024255"/>
-    </inertial>
-    <visual>
-      <origin xyz="0 0 0" rpy="0 0 0"/>
-      <geometry>
-        <mesh filename="package://drobot_description/meshes/right_side_frame.STL"/>
-      </geometry>
+      <origin xyz="-0.0016945696607339 0.00768032725914354 0.0578233422450269" rpy="0 0 0"/>
+      <mass value="0.385275324463581"/>
+      <inertia ixx="0.000226753304752499" ixy="-1.11398827218514E-05" ixz="6.22551133000347E-06"
+               iyy="0.00238329526316141" iyz="-5.33911597507339E-05" izz="0.00245899243822558"/>
+    </inertial>
+    <visual>
+      <origin xyz="0 0 0" rpy="0 0 0"/>
+      <geometry><mesh filename="package://drobot_description/meshes/right_side_frame.STL"/></geometry>
       <material name="frame_color"/>
     </visual>
-  </link>
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
File: src/drobot_description/urdf/gazebo.xacro (robot description, xacro)
@@ -12,18 +12,18 @@
     </plugin>
   </gazebo>
-  <!-- Diff Drive (cmd_vel only, odom disabled — wheel axes are mixed ±Z) -->
+  <!-- Diff Drive -->
   <gazebo>
     <plugin filename="gz-sim-diff-drive-system"
             name="gz::sim::systems::DiffDrive">
-      <left_joint>con_lf_wheel</left_joint>
-      <left_joint>con_lr_wheel</left_joint>
-      <right_joint>con_rf_wheel</right_joint>
-      <right_joint>con_rr_wheel</right_joint>
-      <wheel_separation>0.364</wheel_separation>
+      <left_joint>lf_wheel_con</left_joint>
+      <left_joint>lr_wheel_con</left_joint>
+      <right_joint>rf_wheel_con</right_joint>
+      <right_joint>rr_wheel_con</right_joint>
+      <wheel_separation>0.35</wheel_separation>  <!-- 0.298→0.35: 회전토크 소폭 증가 -->
       <wheel_radius>0.112</wheel_radius>
       <topic>/cmd_vel</topic>
     </plugin>
   </gazebo>
-  <!-- Odometry from model pose (avoids wheel axis sign issue) -->
+  <!-- Odometry from model pose -->
   <gazebo>
     <plugin filename="gz-sim-odometry-publisher-system"
@@ -35,51 +35,10 @@
     </plugin>
   </gazebo>
-  <!-- ========== ARM POSITION CONTROLLERS ========== -->
-  <!-- All arms use same topic /drobot/arm_cmd for synchronized movement -->
-  <gazebo>
-    <plugin filename="gz-sim-joint-position-controller-system"
-            name="gz::sim::systems::JointPositionController">
-      <joint_name>rev_lf_arm</joint_name>
-      <topic>/drobot/arm_cmd</topic>
-      <p_gain>1000</p_gain>
-      <i_gain>100</i_gain>
-      <d_gain>100</d_gain>
-    </plugin>
-  </gazebo>
-  <gazebo>
-    <plugin filename="gz-sim-joint-position-controller-system"
-            name="gz::sim::systems::JointPositionController">
-      <joint_name>rev_lr_arm</joint_name>
-      <topic>/drobot/arm_cmd</topic>
-      <p_gain>1000</p_gain>
-      <i_gain>100</i_gain>
-      <d_gain>100</d_gain>
-    </plugin>
-  </gazebo>
-  <gazebo>
-    <plugin filename="gz-sim-joint-position-controller-system"
-            name="gz::sim::systems::JointPositionController">
-      <joint_name>rev_rf_arm</joint_name>
-      <topic>/drobot/arm_cmd</topic>
-      <p_gain>1000</p_gain>
-      <i_gain>100</i_gain>
-      <d_gain>100</d_gain>
-    </plugin>
-  </gazebo>
-  <gazebo>
-    <plugin filename="gz-sim-joint-position-controller-system"
-            name="gz::sim::systems::JointPositionController">
-      <joint_name>rev_rr_arm</joint_name>
-      <topic>/drobot/arm_cmd</topic>
-      <p_gain>1000</p_gain>
-      <i_gain>100</i_gain>
-      <d_gain>100</d_gain>
-    </plugin>
-  </gazebo>
+  <!-- ARM: held by extreme damping+friction (revolute for future terrain mode) -->
   <!-- ========== 2D LIDAR ========== -->
-  <gazebo reference="lidar_link">
+  <gazebo reference="lidar">
     <sensor name="lidar" type="gpu_lidar">
       <topic>/scan</topic>
-      <gz_frame_id>lidar_link</gz_frame_id>
+      <gz_frame_id>lidar</gz_frame_id>
       <update_rate>10</update_rate>
       <always_on>true</always_on>
@@ -124,8 +83,8 @@
   </gazebo>
   <!-- ========== CAMERA ========== -->
-  <gazebo reference="camera_link">
+  <gazebo reference="camera">
     <sensor name="camera" type="camera">
       <topic>/camera/image_raw</topic>
-      <gz_frame_id>camera_link</gz_frame_id>
+      <gz_frame_id>camera</gz_frame_id>
       <update_rate>15</update_rate>
       <always_on>true</always_on>
@@ -148,20 +107,20 @@
   <gazebo reference="left_front_wheel">
     <collision><surface>
-      <friction><ode><mu>1.0</mu><mu2>0.5</mu2></ode></friction>
+      <friction><ode><mu>1.0</mu><mu2>0.15</mu2></ode></friction>
     </surface></collision>
   </gazebo>
   <gazebo reference="right_front_wheel">
     <collision><surface>
-      <friction><ode><mu>1.0</mu><mu2>0.5</mu2></ode></friction>
+      <friction><ode><mu>1.0</mu><mu2>0.15</mu2></ode></friction>
     </surface></collision>
   </gazebo>
   <gazebo reference="left_rear_wheel">
     <collision><surface>
-      <friction><ode><mu>1.0</mu><mu2>0.5</mu2></ode></friction>
+      <friction><ode><mu>1.0</mu><mu2>0.15</mu2></ode></friction>
     </surface></collision>
   </gazebo>
   <gazebo reference="right_rear_wheel">
     <collision><surface>
-      <friction><ode><mu>1.0</mu><mu2>0.5</mu2></ode></friction>
+      <friction><ode><mu>1.0</mu><mu2>0.15</mu2></ode></friction>
     </surface></collision>
   </gazebo>
