Commit message: Fix wheel rotation asymmetry and tune navigation parameters
- Wheel collision: cylinder → STL mesh (fixes left/right rotation asymmetry)
- Arm joint angles: exact π, π/2 values, mass/inertia equalized
- Gazebo: mu2=0.15, wheel_separation=0.35
- Nav2: RotationShimController for heading alignment before path following
- Nav2: DWB forward-only (min_vel_x=0.0), oscillation critic added
- Nav2: reduced footprint/inflation for narrow passage navigation
- Nav2: global replan rate 0.5→1.0Hz, costmap update 2→5Hz
- Safety: COLLISION_STOP_DIST 0.40→0.25m

Co-Authored-By: Claude Opus 4.6 <noreply@anthropic.com>

File: src/drobot_description/urdf/ros2_control.xacro (robot description, xacro)
@@ -5,15 +5,19 @@
       <hardware><plugin>gz_ros2_control/GazeboSimSystem</plugin></hardware>
     </xacro:if>
-    <joint name="rev_lf_arm">
-      <command_interface name="position">
-        <param name="min">0.0</param><param name="max">1.5708</param>
-      </command_interface>
-      <state_interface name="position"/><state_interface name="velocity"/>
-    </joint>
-    <joint name="con_lf_wheel">
+    <!-- Arm joints are fixed for rover mode -->
+    <!-- Wheel joints (velocity control) -->
+    <joint name="lf_wheel_con">
       <command_interface name="velocity"/>
       <state_interface name="position"/><state_interface name="velocity"/>
     </joint>
-    <joint name="con_rf_wheel">
+    <joint name="lr_wheel_con">
+      <command_interface name="velocity"/>
+      <state_interface name="position"/><state_interface name="velocity"/>
+    </joint>
+    <joint name="rf_wheel_con">
+      <command_interface name="velocity"/>
+      <state_interface name="position"/><state_interface name="velocity"/>
+    </joint>
+    <joint name="rr_wheel_con">
       <command_interface name="velocity"/>
       <state_interface name="position"/><state_interface name="velocity"/>
