Commit message: perception 파라미터화 (conf_threshold, post_filter_conf, max_detect_distance) 및 .DS_Store gitignore 추가
Co-Authored-By: Claude Opus 4.6 <noreply@anthropic.com>

File: ros2_ws/src/drobot_description/urdf/drobot.urdf.xacro (robot description, xacro)
@@ -127,6 +127,6 @@
     <child link="left_front_arm"/>
     <axis xyz="-1 0 0"/>
-    <limit lower="0" upper="1.5708" effort="100" velocity="2"/>
-    <dynamics damping="500.0" friction="50.0"/>
+    <limit lower="0" upper="1.5708" effort="2.45" velocity="8.06"/>
+    <dynamics damping="0.5" friction="0.1"/>
   </joint>
   <!-- ==================== LEFT SIDE FRAME ==================== -->
@@ -233,6 +233,6 @@
     <child link="left_rear_arm"/>
     <axis xyz="-1 0 0"/>
-    <limit lower="0" upper="1.5708" effort="100" velocity="2"/>
-    <dynamics damping="500.0" friction="50.0"/>
+    <limit lower="0" upper="1.5708" effort="2.45" velocity="8.06"/>
+    <dynamics damping="0.5" friction="0.1"/>
   </joint>
   <!-- ==================== RIGHT FRONT ARM ==================== -->
@@ -259,6 +259,6 @@
     <child link="right_front_arm"/>
     <axis xyz="1 0 0"/>
-    <limit lower="0" upper="1.5708" effort="100" velocity="2"/>
-    <dynamics damping="500.0" friction="50.0"/>
+    <limit lower="0" upper="1.5708" effort="2.45" velocity="8.06"/>
+    <dynamics damping="0.5" friction="0.1"/>
   </joint>
   <!-- ==================== RIGHT SIDE FRAME ==================== -->
@@ -361,6 +361,6 @@
     <child link="right_rear_arm"/>
     <axis xyz="-1 0 0"/>
-    <limit lower="0" upper="1.5708" effort="100" velocity="2"/>
-    <dynamics damping="500.0" friction="50.0"/>
+    <limit lower="0" upper="1.5708" effort="2.45" velocity="8.06"/>
+    <dynamics damping="0.5" friction="0.1"/>
   </joint>
   <!-- ==================== ROS2 CONTROL ==================== -->

File: ros2_ws/src/drobot_description/urdf/gazebo.xacro (robot description, xacro)
@@ -35,5 +35,62 @@
     </plugin>
   </gazebo>
-  <!-- ARM: held by extreme damping+friction (revolute for future terrain mode) -->
+  <!-- ========== ARM JOINT POSITION CONTROLLERS ========== -->
+  <!-- Servo spec: 25kg·cm (2.45 N·m), 0.13s/60° @ 6.8V -->
+  <gazebo>
+    <plugin filename="gz-sim-joint-position-controller-system"
+            name="gz::sim::systems::JointPositionController">
+      <joint_name>lf_arm_rev</joint_name>
+      <topic>/model/drobot/joint/lf_arm_rev/cmd_pos</topic>
+      <p_gain>5.0</p_gain>
+      <i_gain>0.5</i_gain>
+      <d_gain>1.0</d_gain>
+      <i_max>1.0</i_max>
+      <i_min>-1.0</i_min>
+      <cmd_max>2.45</cmd_max>
+      <cmd_min>-2.45</cmd_min>
+    </plugin>
+  </gazebo>
+  <gazebo>
+    <plugin filename="gz-sim-joint-position-controller-system"
+            name="gz::sim::systems::JointPositionController">
+      <joint_name>lr_arm_rev</joint_name>
+      <topic>/model/drobot/joint/lr_arm_rev/cmd_pos</topic>
+      <p_gain>5.0</p_gain>
+      <i_gain>0.5</i_gain>
+      <d_gain>1.0</d_gain>
+      <i_max>1.0</i_max>
+      <i_min>-1.0</i_min>
+      <cmd_max>2.45</cmd_max>
+      <cmd_min>-2.45</cmd_min>
+    </plugin>
+  </gazebo>
+  <gazebo>
+    <plugin filename="gz-sim-joint-position-controller-system"
+            name="gz::sim::systems::JointPositionController">
+      <joint_name>rf_arm_rev</joint_name>
+      <topic>/model/drobot/joint/rf_arm_rev/cmd_pos</topic>
+      <p_gain>5.0</p_gain>
+      <i_gain>0.5</i_gain>
+      <d_gain>1.0</d_gain>
+      <i_max>1.0</i_max>
+      <i_min>-1.0</i_min>
+      <cmd_max>2.45</cmd_max>
+      <cmd_min>-2.45</cmd_min>
+    </plugin>
+  </gazebo>
+  <gazebo>
+    <plugin filename="gz-sim-joint-position-controller-system"
+            name="gz::sim::systems::JointPositionController">
+      <joint_name>rr_arm_rev</joint_name>
+      <topic>/model/drobot/joint/rr_arm_rev/cmd_pos</topic>
+      <p_gain>5.0</p_gain>
+      <i_gain>0.5</i_gain>
+      <d_gain>1.0</d_gain>
+      <i_max>1.0</i_max>
+      <i_min>-1.0</i_min>
+      <cmd_max>2.45</cmd_max>
+      <cmd_min>-2.45</cmd_min>
+    </plugin>
+  </gazebo>
   <!-- ========== 2D LIDAR ========== -->
   <gazebo reference="lidar">
