Commit message: lidar범위 수정 및 rr arm axis수정

File: ros2_ws/src/drobot_description/urdf/drobot.urdf.xacro (robot description, xacro)
@@ -360,5 +360,5 @@
     <parent link="base_link"/>
     <child link="right_rear_arm"/>
-    <axis xyz="-1 0 0"/>
+    <axis xyz="1 0 0"/>
     <limit lower="0" upper="1.5708" effort="2.45" velocity="8.06"/>
     <dynamics damping="0.5" friction="0.1"/>

File: ros2_ws/src/drobot_description/urdf/gazebo.xacro (robot description, xacro)
@@ -111,5 +111,5 @@
         </scan>
         <range>
-          <min>0.15</min>
+          <min>0.25</min>
           <max>12.0</max>
           <resolution>0.01</resolution>

Commit message: effort, pid값 수정

File: ros2_ws/src/drobot_description/urdf/drobot.urdf.xacro (robot description, xacro)
@@ -127,6 +127,6 @@
     <child link="left_front_arm"/>
     <axis xyz="-1 0 0"/>
-    <limit lower="0" upper="1.5708" effort="2.45" velocity="8.06"/>
-    <dynamics damping="0.5" friction="0.1"/>
+    <limit lower="0" upper="1.5708" effort="5.0" velocity="0.5"/>
+    <dynamics damping="3.0" friction="1.0"/>
   </joint>
   <!-- ==================== LEFT SIDE FRAME ==================== -->
@@ -233,6 +233,6 @@
     <child link="left_rear_arm"/>
     <axis xyz="-1 0 0"/>
-    <limit lower="0" upper="1.5708" effort="2.45" velocity="8.06"/>
-    <dynamics damping="0.5" friction="0.1"/>
+    <limit lower="0" upper="1.5708" effort="5.0" velocity="0.5"/>
+    <dynamics damping="3.0" friction="1.0"/>
   </joint>
   <!-- ==================== RIGHT FRONT ARM ==================== -->
@@ -259,6 +259,6 @@
     <child link="right_front_arm"/>
     <axis xyz="1 0 0"/>
-    <limit lower="0" upper="1.5708" effort="2.45" velocity="8.06"/>
-    <dynamics damping="0.5" friction="0.1"/>
+    <limit lower="0" upper="1.5708" effort="5.0" velocity="0.5"/>
+    <dynamics damping="3.0" friction="1.0"/>
   </joint>
   <!-- ==================== RIGHT SIDE FRAME ==================== -->
@@ -361,6 +361,6 @@
     <child link="right_rear_arm"/>
     <axis xyz="1 0 0"/>
-    <limit lower="0" upper="1.5708" effort="2.45" velocity="8.06"/>
-    <dynamics damping="0.5" friction="0.1"/>
+    <limit lower="0" upper="1.5708" effort="5.0" velocity="0.5"/>
+    <dynamics damping="3.0" friction="1.0"/>
   </joint>
   <!-- ==================== ROS2 CONTROL ==================== -->

File: ros2_ws/src/drobot_description/urdf/gazebo.xacro (robot description, xacro)
@@ -42,11 +42,11 @@
       <joint_name>lf_arm_rev</joint_name>
       <topic>/model/drobot/joint/lf_arm_rev/cmd_pos</topic>
-      <p_gain>5.0</p_gain>
+      <p_gain>10.0</p_gain>
       <i_gain>0.5</i_gain>
       <d_gain>1.0</d_gain>
       <i_max>1.0</i_max>
       <i_min>-1.0</i_min>
-      <cmd_max>2.45</cmd_max>
-      <cmd_min>-2.45</cmd_min>
+      <cmd_max>5.0</cmd_max>
+      <cmd_min>-5.0</cmd_min>
     </plugin>
   </gazebo>
@@ -56,11 +56,11 @@
       <joint_name>lr_arm_rev</joint_name>
       <topic>/model/drobot/joint/lr_arm_rev/cmd_pos</topic>
-      <p_gain>5.0</p_gain>
+      <p_gain>10.0</p_gain>
       <i_gain>0.5</i_gain>
       <d_gain>1.0</d_gain>
       <i_max>1.0</i_max>
       <i_min>-1.0</i_min>
-      <cmd_max>2.45</cmd_max>
-      <cmd_min>-2.45</cmd_min>
+      <cmd_max>5.0</cmd_max>
+      <cmd_min>-5.0</cmd_min>
     </plugin>
   </gazebo>
@@ -70,11 +70,11 @@
       <joint_name>rf_arm_rev</joint_name>
       <topic>/model/drobot/joint/rf_arm_rev/cmd_pos</topic>
-      <p_gain>5.0</p_gain>
+      <p_gain>10.0</p_gain>
       <i_gain>0.5</i_gain>
       <d_gain>1.0</d_gain>
       <i_max>1.0</i_max>
       <i_min>-1.0</i_min>
-      <cmd_max>2.45</cmd_max>
-      <cmd_min>-2.45</cmd_min>
+      <cmd_max>5.0</cmd_max>
+      <cmd_min>-5.0</cmd_min>
     </plugin>
   </gazebo>
@@ -84,11 +84,11 @@
       <joint_name>rr_arm_rev</joint_name>
       <topic>/model/drobot/joint/rr_arm_rev/cmd_pos</topic>
-      <p_gain>5.0</p_gain>
+      <p_gain>10.0</p_gain>
       <i_gain>0.5</i_gain>
       <d_gain>1.0</d_gain>
       <i_max>1.0</i_max>
       <i_min>-1.0</i_min>
-      <cmd_max>2.45</cmd_max>
-      <cmd_min>-2.45</cmd_min>
+      <cmd_max>5.0</cmd_max>
+      <cmd_min>-5.0</cmd_min>
     </plugin>
   </gazebo>

Commit message: revise software

File: ros2_ws/src/drobot_description/urdf/drobot.urdf.xacro (robot description, xacro)
@@ -127,6 +127,6 @@
     <child link="left_front_arm"/>
     <axis xyz="-1 0 0"/>
-    <limit lower="0" upper="1.5708" effort="5.0" velocity="0.5"/>
-    <dynamics damping="3.0" friction="1.0"/>
+    <limit lower="0" upper="1.5708" effort="7.0" velocity="0.5"/>
+    <dynamics damping="3.0" friction="3.0"/>
   </joint>
   <!-- ==================== LEFT SIDE FRAME ==================== -->
@@ -233,6 +233,6 @@
     <child link="left_rear_arm"/>
     <axis xyz="-1 0 0"/>
-    <limit lower="0" upper="1.5708" effort="5.0" velocity="0.5"/>
-    <dynamics damping="3.0" friction="1.0"/>
+    <limit lower="0" upper="1.5708" effort="7.0" velocity="0.5"/>
+    <dynamics damping="3.0" friction="3.0"/>
   </joint>
   <!-- ==================== RIGHT FRONT ARM ==================== -->
@@ -259,6 +259,6 @@
     <child link="right_front_arm"/>
     <axis xyz="1 0 0"/>
-    <limit lower="0" upper="1.5708" effort="5.0" velocity="0.5"/>
-    <dynamics damping="3.0" friction="1.0"/>
+    <limit lower="0" upper="1.5708" effort="7.0" velocity="0.5"/>
+    <dynamics damping="3.0" friction="3.0"/>
   </joint>
   <!-- ==================== RIGHT SIDE FRAME ==================== -->
@@ -361,6 +361,6 @@
     <child link="right_rear_arm"/>
     <axis xyz="1 0 0"/>
-    <limit lower="0" upper="1.5708" effort="5.0" velocity="0.5"/>
-    <dynamics damping="3.0" friction="1.0"/>
+    <limit lower="0" upper="1.5708" effort="7.0" velocity="0.5"/>
+    <dynamics damping="3.0" friction="3.0"/>
   </joint>
   <!-- ==================== ROS2 CONTROL ==================== -->

File: ros2_ws/src/drobot_description/urdf/gazebo.xacro (robot description, xacro)
@@ -47,6 +47,6 @@
       <i_max>1.0</i_max>
       <i_min>-1.0</i_min>
-      <cmd_max>5.0</cmd_max>
-      <cmd_min>-5.0</cmd_min>
+      <cmd_max>7.0</cmd_max>
+      <cmd_min>-7.0</cmd_min>
     </plugin>
   </gazebo>
@@ -61,6 +61,6 @@
       <i_max>1.0</i_max>
       <i_min>-1.0</i_min>
-      <cmd_max>5.0</cmd_max>
-      <cmd_min>-5.0</cmd_min>
+      <cmd_max>7.0</cmd_max>
+      <cmd_min>-7.0</cmd_min>
     </plugin>
   </gazebo>
@@ -75,6 +75,6 @@
       <i_max>1.0</i_max>
       <i_min>-1.0</i_min>
-      <cmd_max>5.0</cmd_max>
-      <cmd_min>-5.0</cmd_min>
+      <cmd_max>7.0</cmd_max>
+      <cmd_min>-7.0</cmd_min>
     </plugin>
   </gazebo>
@@ -89,6 +89,6 @@
       <i_max>1.0</i_max>
       <i_min>-1.0</i_min>
-      <cmd_max>5.0</cmd_max>
-      <cmd_min>-5.0</cmd_min>
+      <cmd_max>7.0</cmd_max>
+      <cmd_min>-7.0</cmd_min>
     </plugin>
   </gazebo>
@@ -111,5 +111,5 @@
         </scan>
         <range>
-          <min>0.25</min>
+          <min>0.5</min>
           <max>12.0</max>
           <resolution>0.01</resolution>

Commit message: ffinn

File: ros2_ws/src/drobot_description/urdf/drobot.urdf.xacro (robot description, xacro)
@@ -127,6 +127,6 @@
     <child link="left_front_arm"/>
     <axis xyz="-1 0 0"/>
-    <limit lower="0" upper="1.5708" effort="7.0" velocity="0.5"/>
-    <dynamics damping="3.0" friction="3.0"/>
+    <limit lower="0" upper="1.5708" effort="14.0" velocity="0.5"/>
+    <dynamics damping="4.0" friction="5.0"/>
   </joint>
   <!-- ==================== LEFT SIDE FRAME ==================== -->
@@ -233,5 +233,5 @@
     <child link="left_rear_arm"/>
     <axis xyz="-1 0 0"/>
-    <limit lower="0" upper="1.5708" effort="7.0" velocity="0.5"/>
+    <limit lower="0" upper="1.5708" effort="14.0" velocity="0.5"/>
     <dynamics damping="3.0" friction="3.0"/>
   </joint>
@@ -259,6 +259,6 @@
     <child link="right_front_arm"/>
     <axis xyz="1 0 0"/>
-    <limit lower="0" upper="1.5708" effort="7.0" velocity="0.5"/>
-    <dynamics damping="3.0" friction="3.0"/>
+    <limit lower="0" upper="1.5708" effort="14.0" velocity="0.5"/>
+    <dynamics damping="4.0" friction="5.0"/>
   </joint>
   <!-- ==================== RIGHT SIDE FRAME ==================== -->
@@ -361,5 +361,5 @@
     <child link="right_rear_arm"/>
     <axis xyz="1 0 0"/>
-    <limit lower="0" upper="1.5708" effort="7.0" velocity="0.5"/>
+    <limit lower="0" upper="1.5708" effort="14.0" velocity="0.5"/>
     <dynamics damping="3.0" friction="3.0"/>
   </joint>

File: ros2_ws/src/drobot_description/urdf/gazebo.xacro (robot description, xacro)
@@ -42,11 +42,11 @@
       <joint_name>lf_arm_rev</joint_name>
       <topic>/model/drobot/joint/lf_arm_rev/cmd_pos</topic>
-      <p_gain>10.0</p_gain>
-      <i_gain>0.5</i_gain>
-      <d_gain>1.0</d_gain>
-      <i_max>1.0</i_max>
-      <i_min>-1.0</i_min>
-      <cmd_max>7.0</cmd_max>
-      <cmd_min>-7.0</cmd_min>
+      <p_gain>20.0</p_gain>
+      <i_gain>1.0</i_gain>
+      <d_gain>2.0</d_gain>
+      <i_max>5.0</i_max>
+      <i_min>-5.0</i_min>
+      <cmd_max>14.0</cmd_max>
+      <cmd_min>-14.0</cmd_min>
     </plugin>
   </gazebo>
@@ -56,11 +56,11 @@
       <joint_name>lr_arm_rev</joint_name>
       <topic>/model/drobot/joint/lr_arm_rev/cmd_pos</topic>
-      <p_gain>10.0</p_gain>
-      <i_gain>0.5</i_gain>
-      <d_gain>1.0</d_gain>
-      <i_max>1.0</i_max>
-      <i_min>-1.0</i_min>
-      <cmd_max>7.0</cmd_max>
-      <cmd_min>-7.0</cmd_min>
+      <p_gain>20.0</p_gain>
+      <i_gain>1.0</i_gain>
+      <d_gain>2.0</d_gain>
+      <i_max>5.0</i_max>
+      <i_min>-5.0</i_min>
+      <cmd_max>14.0</cmd_max>
+      <cmd_min>-14.0</cmd_min>
     </plugin>
   </gazebo>
@@ -70,11 +70,11 @@
       <joint_name>rf_arm_rev</joint_name>
       <topic>/model/drobot/joint/rf_arm_rev/cmd_pos</topic>
-      <p_gain>10.0</p_gain>
-      <i_gain>0.5</i_gain>
-      <d_gain>1.0</d_gain>
-      <i_max>1.0</i_max>
-      <i_min>-1.0</i_min>
-      <cmd_max>7.0</cmd_max>
-      <cmd_min>-7.0</cmd_min>
+      <p_gain>20.0</p_gain>
+      <i_gain>1.0</i_gain>
+      <d_gain>2.0</d_gain>
+      <i_max>5.0</i_max>
+      <i_min>-5.0</i_min>
+      <cmd_max>14.0</cmd_max>
+      <cmd_min>-14.0</cmd_min>
     </plugin>
   </gazebo>
@@ -84,11 +84,11 @@
       <joint_name>rr_arm_rev</joint_name>
       <topic>/model/drobot/joint/rr_arm_rev/cmd_pos</topic>
-      <p_gain>10.0</p_gain>
-      <i_gain>0.5</i_gain>
-      <d_gain>1.0</d_gain>
-      <i_max>1.0</i_max>
-      <i_min>-1.0</i_min>
-      <cmd_max>7.0</cmd_max>
-      <cmd_min>-7.0</cmd_min>
+      <p_gain>20.0</p_gain>
+      <i_gain>1.0</i_gain>
+      <d_gain>2.0</d_gain>
+      <i_max>5.0</i_max>
+      <i_min>-5.0</i_min>
+      <cmd_max>14.0</cmd_max>
+      <cmd_min>-14.0</cmd_min>
     </plugin>
   </gazebo>
@@ -162,20 +162,20 @@
   <gazebo reference="left_front_wheel">
     <collision><surface>
-      <friction><ode><mu>1.0</mu><mu2>0.15</mu2></ode></friction>
+      <friction><ode><mu>1.0</mu><mu2>0.3</mu2><fdir1>1 0 0</fdir1></ode></friction>
     </surface></collision>
   </gazebo>
   <gazebo reference="right_front_wheel">
     <collision><surface>
-      <friction><ode><mu>1.0</mu><mu2>0.15</mu2></ode></friction>
+      <friction><ode><mu>1.0</mu><mu2>0.3</mu2><fdir1>1 0 0</fdir1></ode></friction>
     </surface></collision>
   </gazebo>
   <gazebo reference="left_rear_wheel">
     <collision><surface>
-      <friction><ode><mu>1.0</mu><mu2>0.15</mu2></ode></friction>
+      <friction><ode><mu>1.0</mu><mu2>0.3</mu2><fdir1>1 0 0</fdir1></ode></friction>
     </surface></collision>
   </gazebo>
   <gazebo reference="right_rear_wheel">
     <collision><surface>
-      <friction><ode><mu>1.0</mu><mu2>0.15</mu2></ode></friction>
+      <friction><ode><mu>1.0</mu><mu2>0.3</mu2><fdir1>1 0 0</fdir1></ode></friction>
     </surface></collision>
   </gazebo>

Commit message: fixed left rear arm

File: ros2_ws/src/drobot_description/urdf/drobot.urdf.xacro (robot description, xacro)
@@ -213,5 +213,5 @@
   <link name="left_rear_arm">
     <inertial>
-      <origin xyz="-0.000999999999999908 0.00407538533818062 -0.000143536147134726" rpy="0 0 0"/>
+      <origin xyz="0.018998 -0.000534 0.112534" rpy="0 0 0"/>
       <mass value="0.123064431731573"/>
       <inertia ixx="0.000135741612972814" ixy="6.13644622591408E-06" ixz="-3.91949328277525E-06"
@@ -219,15 +219,15 @@
     </inertial>
     <visual>
-      <origin xyz="0 0 0" rpy="0 0 0"/>
+      <origin xyz="0 -0.003671 -0.216881" rpy="0 0 0"/>
       <geometry><mesh filename="package://drobot_description/meshes/left_rear_arm.STL"/></geometry>
       <material name="arm_color"/>
     </visual>
-    <collision>
-      <origin xyz="0 0 0" rpy="0 0 0"/>
+    <!-- <collision>
+      <origin xyz="0 -0.003671 -0.216881" rpy="0 0 0"/>
       <geometry><mesh filename="package://drobot_description/meshes/left_rear_arm.STL"/></geometry>
-    </collision>
+    </collision> -->
   </link>
   <joint name="lr_arm_rev" type="revolute">
-    <origin xyz="0.001 -0.19728 0.21693" rpy="1.5708 0 3.1416"/>
+    <origin xyz="0.001 0.022 0.240" rpy="1.5708 0 3.1416"/>
     <parent link="base_link"/>
     <child link="left_rear_arm"/>
@@ -341,5 +341,5 @@
   <link name="right_rear_arm">
     <inertial>
-      <origin xyz="0.0954185913955707 -0.00383727803839913 0.136265758086407" rpy="0 0 0"/>
+      <origin xyz="-0.072133 0.029001 -0.051593" rpy="0 0 0"/>
       <mass value="0.123064431731573"/>
       <inertia ixx="0.000135741612972814" ixy="6.13644622591408E-06" ixz="-3.91949328277525E-06"
@@ -347,15 +347,16 @@
     </inertial>
     <visual>
-      <origin xyz="0 0 0" rpy="0 0 0"/>
+      <origin xyz="0 -0.002488 -0.180993" rpy="0 0 0"/>
       <geometry><mesh filename="package://drobot_description/meshes/right_rear_arm.STL"/></geometry>
       <material name="arm_color"/>
     </visual>
-    <collision>
-      <origin xyz="0 0 0" rpy="0 0 0"/>
+    <!-- deleted temporarly-->
+    <!-- <collision>
+      <origin xyz="0 -0.002488 -0.180993" rpy="0 0 0"/>
       <geometry><mesh filename="package://drobot_description/meshes/right_rear_arm.STL"/></geometry>
-    </collision>
+    </collision> -->
   </link>
   <joint name="rr_arm_rev" type="revolute">
-    <origin xyz="0.002 -0.1975 0.221" rpy="1.5708 0 3.1416"/>
+    <origin xyz="0.001 -0.023 0.27" rpy="1.5708 0 3.1416"/>
     <parent link="base_link"/>
     <child link="right_rear_arm"/>

Commit message: fixed rrm

File: ros2_ws/src/drobot_description/urdf/drobot.urdf.xacro (robot description, xacro)
@@ -219,5 +219,5 @@
     </inertial>
     <visual>
-      <origin xyz="0 -0.003671 -0.216881" rpy="0 0 0"/>
+      <origin xyz="0 -0.023671 -0.216881" rpy="0 0 0"/>
       <geometry><mesh filename="package://drobot_description/meshes/left_rear_arm.STL"/></geometry>
       <material name="arm_color"/>
@@ -341,5 +341,5 @@
   <link name="right_rear_arm">
     <inertial>
-      <origin xyz="-0.072133 0.029001 -0.051593" rpy="0 0 0"/>
+      <origin xyz="-0.072133 0.029001 -0.151593" rpy="0 0 0"/>
       <mass value="0.123064431731573"/>
       <inertia ixx="0.000135741612972814" ixy="6.13644622591408E-06" ixz="-3.91949328277525E-06"
@@ -347,5 +347,5 @@
     </inertial>
     <visual>
-      <origin xyz="0 -0.002488 -0.180993" rpy="0 0 0"/>
+      <origin xyz="0 -0.022488 -0.180993" rpy="0 0 0"/>
       <geometry><mesh filename="package://drobot_description/meshes/right_rear_arm.STL"/></geometry>
       <material name="arm_color"/>
@@ -358,5 +358,5 @@
   </link>
   <joint name="rr_arm_rev" type="revolute">
-    <origin xyz="0.001 -0.023 0.27" rpy="1.5708 0 3.1416"/>
+    <origin xyz="0.001 -0.023 0.245" rpy="1.5708 0 3.1416"/>
     <parent link="base_link"/>
     <child link="right_rear_arm"/>

Commit message: smooth morphing

File: ros2_ws/src/drobot_description/urdf/drobot.urdf.xacro (robot description, xacro)
@@ -107,5 +107,5 @@
   <link name="left_front_arm">
     <inertial>
-      <origin xyz="0.018998 -0.000534 0.112534" rpy="0 0 0"/>
+      <origin xyz="0.018998 0.04 0.112534" rpy="0 0 0"/>
       <mass value="0.123064431731573"/>
       <inertia ixx="0.000135741612972814" ixy="6.13644622591408E-06" ixz="-3.91949328277525E-06"
@@ -113,15 +113,15 @@
     </inertial>
     <visual>
-      <origin xyz="0 -0.003671 -0.216881" rpy="0 0 0"/>
+      <origin xyz="0 0 -0.216881" rpy="0 0 0"/>
       <geometry><mesh filename="package://drobot_description/meshes/left_front_arm.STL"/></geometry>
       <material name="arm_color"/>
     </visual>
     <collision>
-      <origin xyz="0 -0.003671 -0.216881" rpy="0 0 0"/>
+      <origin xyz="0 0 -0.216881" rpy="0 0 0"/>
       <geometry><mesh filename="package://drobot_description/meshes/left_front_arm.STL"/></geometry>
     </collision>
   </link>
   <joint name="lf_arm_rev" type="revolute">
-    <origin xyz="0.001 0.022 0.240" rpy="3.1416 0 3.1416"/>
+    <origin xyz="0.001 0.024 0.240" rpy="3.1416 0 3.1416"/>
     <parent link="base_link"/>
     <child link="left_front_arm"/>
@@ -219,5 +219,5 @@
     </inertial>
     <visual>
-      <origin xyz="0 -0.023671 -0.216881" rpy="0 0 0"/>
+      <origin xyz="0 -0.022671 -0.216881" rpy="0 0 0"/>
       <geometry><mesh filename="package://drobot_description/meshes/left_rear_arm.STL"/></geometry>
       <material name="arm_color"/>
@@ -229,5 +229,5 @@
   </link>
   <joint name="lr_arm_rev" type="revolute">
-    <origin xyz="0.001 0.022 0.240" rpy="1.5708 0 3.1416"/>
+    <origin xyz="0.001 0.024 0.240" rpy="1.5708 0 3.1416"/>
     <parent link="base_link"/>
     <child link="left_rear_arm"/>
@@ -239,5 +239,5 @@
   <link name="right_front_arm">
     <inertial>
-      <origin xyz="-0.072133 0.029001 -0.051593" rpy="0 0 0"/>
+      <origin xyz="-0.072133 0.017001 -0.051593" rpy="0 0 0"/>
       <mass value="0.123064431731573"/>
       <inertia ixx="0.000135741612972814" ixy="6.13644622591408E-06" ixz="-3.91949328277525E-06"
@@ -245,15 +245,15 @@
     </inertial>
     <visual>
-      <origin xyz="0 -0.002488 -0.180993" rpy="0 0 0"/>
+      <origin xyz="0 -0.002488 -0.175993" rpy="0 0 0"/>
       <geometry><mesh filename="package://drobot_description/meshes/right_front_arm.STL"/></geometry>
       <material name="arm_color"/>
     </visual>
     <collision>
-      <origin xyz="0 -0.002488 -0.180993" rpy="0 0 0"/>
+      <origin xyz="0 -0.002488 -0.175993" rpy="0 0 0"/>
       <geometry><mesh filename="package://drobot_description/meshes/right_front_arm.STL"/></geometry>
     </collision>
   </link>
   <joint name="rf_arm_rev" type="revolute">
-    <origin xyz="0.001 -0.023 0.245" rpy="0 0 3.1416"/>
+    <origin xyz="0.001 -0.025 0.249" rpy="0 0 3.1416"/>
     <parent link="base_link"/>
     <child link="right_front_arm"/>
@@ -341,5 +341,5 @@
   <link name="right_rear_arm">
     <inertial>
-      <origin xyz="-0.072133 0.029001 -0.151593" rpy="0 0 0"/>
+      <origin xyz="-0.072133 0.027001 -0.151593" rpy="0 0 0"/>
       <mass value="0.123064431731573"/>
       <inertia ixx="0.000135741612972814" ixy="6.13644622591408E-06" ixz="-3.91949328277525E-06"
@@ -347,5 +347,5 @@
     </inertial>
     <visual>
-      <origin xyz="0 -0.022488 -0.180993" rpy="0 0 0"/>
+      <origin xyz="0 -0.022488 -0.175993" rpy="0 0 0"/>
       <geometry><mesh filename="package://drobot_description/meshes/right_rear_arm.STL"/></geometry>
       <material name="arm_color"/>
@@ -358,5 +358,5 @@
   </link>
   <joint name="rr_arm_rev" type="revolute">
-    <origin xyz="0.001 -0.023 0.245" rpy="1.5708 0 3.1416"/>
+    <origin xyz="0.001 -0.025 0.249" rpy="1.5708 0 3.1416"/>
     <parent link="base_link"/>
     <child link="right_rear_arm"/>
