Commit message: Fix new_gazebo joint stability and add joint position controllers

File: ros2_ws/src/drobot_description/urdf_sub/drobotv0.urdf (robot description, URDF)
Before this commit: robot drobotv0, 11 links, 10 joints
Joints:
- removed joint wheejoint_LF
- added joint wheeljoint_LF: type continuous, parent arm_left, child wheel_LF, origin xyz=0.023562 0.08366 -0.059076 rpy=0 0 0, axis 0 0.99994 0.011086, limit lower=-3.14 upper=3.14 effort=1 velocity=1

File: ros2_ws/src/drobot_description/urdf_sub/drobotv0.urdf.xacro (robot description, xacro)
@@ -99,8 +99,9 @@
       xyz="1 0 0" />
     <limit
-      lower="-3.14"
-      upper="3.14"
-      effort="1"
-      velocity="1" />
+      lower="-0.60"
+      upper="0.60"
+      effort="100"
+      velocity="2.0" />
+    <dynamics damping="40.0" friction="8.0" />
   </joint>
   <link
@@ -157,8 +158,9 @@
       xyz="1 0 0" />
     <limit
-      lower="-3.14"
-      upper="3.14"
-      effort="1"
-      velocity="1" />
+      lower="-0.40"
+      upper="0.90"
+      effort="120"
+      velocity="2.0" />
+    <dynamics damping="50.0" friction="10.0" />
   </joint>
   <link
@@ -203,5 +205,5 @@
   </link>
   <joint
-    name="wheejoint_LF"
+    name="wheeljoint_LF"
     type="continuous">
     <origin
@@ -331,12 +333,9 @@
       xyz="-1 0 0" />
     <limit
-      lower="-3.14"
-      upper="3.14"
-      effort="1"
-      velocity="1" />
-    <mimic
-      joint="servo_LF"
-      multiplier="-1"
-      offset="0" />
+      lower="-0.60"
+      upper="0.60"
+      effort="100"
+      velocity="2.0" />
+    <dynamics damping="40.0" friction="8.0" />
   </joint>
   <link
@@ -393,12 +392,9 @@
       xyz="-1 0 0" />
     <limit
-      lower="-3.14"
-      upper="3.14"
-      effort="1"
-      velocity="1" />
-    <mimic
-      joint="servo_LF"
-      multiplier="1"
-      offset="0" />
+      lower="-0.60"
+      upper="0.60"
+      effort="100"
+      velocity="2.0" />
+    <dynamics damping="40.0" friction="8.0" />
   </joint>
   <link
@@ -455,12 +451,9 @@
       xyz="-1 0 0" />
     <limit
-      lower="-3.14"
-      upper="3.14"
-      effort="1"
-      velocity="1" />
-    <mimic
-      joint="armjoint_left"
-      multiplier="1"
-      offset="0" />
+      lower="-0.40"
+      upper="0.90"
+      effort="120"
+      velocity="2.0" />
+    <dynamics damping="50.0" friction="10.0" />
   </joint>
   <link
@@ -633,12 +626,9 @@
       xyz="1 0 0" />
     <limit
-      lower="-3.14"
-      upper="3.14"
-      effort="1"
-      velocity="1" />
-    <mimic
-      joint="servo_RF"
-      multiplier="-1"
-      offset="0" />
+      lower="-0.60"
+      upper="0.60"
+      effort="100"
+      velocity="2.0" />
+    <dynamics damping="40.0" friction="8.0" />
   </joint>
   <!-- Gazebo systems for teleop (/cmd_vel) -->
@@ -664,4 +654,83 @@
     </plugin>
   </gazebo>
+  <!-- Joint position controllers (Gazebo topic control) -->
+  <gazebo>
+    <plugin filename="gz-sim-joint-position-controller-system"
+            name="gz::sim::systems::JointPositionController">
+      <joint_name>servo_LF</joint_name>
+      <topic>/servo_LF/cmd_pos</topic>
+      <initial_position>0.0</initial_position>
+      <p_gain>20.0</p_gain>
+      <i_gain>0.0</i_gain>
+      <d_gain>1.0</d_gain>
+      <cmd_max>200.0</cmd_max>
+      <cmd_min>-200.0</cmd_min>
+    </plugin>
+  </gazebo>
+  <gazebo>
+    <plugin filename="gz-sim-joint-position-controller-system"
+            name="gz::sim::systems::JointPositionController">
+      <joint_name>servo_LR</joint_name>
+      <topic>/servo_LR/cmd_pos</topic>
+      <initial_position>0.0</initial_position>
+      <p_gain>20.0</p_gain>
+      <i_gain>0.0</i_gain>
+      <d_gain>1.0</d_gain>
+      <cmd_max>200.0</cmd_max>
+      <cmd_min>-200.0</cmd_min>
+    </plugin>
+  </gazebo>
+  <gazebo>
+    <plugin filename="gz-sim-joint-position-controller-system"
+            name="gz::sim::systems::JointPositionController">
+      <joint_name>servo_RF</joint_name>
+      <topic>/servo_RF/cmd_pos</topic>
+      <initial_position>0.0</initial_position>
+      <p_gain>20.0</p_gain>
+      <i_gain>0.0</i_gain>
+      <d_gain>1.0</d_gain>
+      <cmd_max>200.0</cmd_max>
+      <cmd_min>-200.0</cmd_min>
+    </plugin>
+  </gazebo>
+  <gazebo>
+    <plugin filename="gz-sim-joint-position-controller-system"
+            name="gz::sim::systems::JointPositionController">
+      <joint_name>servo_RR</joint_name>
+      <topic>/servo_RR/cmd_pos</topic>
+      <initial_position>0.0</initial_position>
+      <p_gain>20.0</p_gain>
+      <i_gain>0.0</i_gain>
+      <d_gain>1.0</d_gain>
+      <cmd_max>200.0</cmd_max>
+      <cmd_min>-200.0</cmd_min>
+    </plugin>
+  </gazebo>
+  <gazebo>
+    <plugin filename="gz-sim-joint-position-controller-system"
+            name="gz::sim::systems::JointPositionController">
+      <joint_name>armjoint_left</joint_name>
+      <topic>/armjoint_left/cmd_pos</topic>
+      <initial_position>0.0</initial_position>
+      <p_gain>20.0</p_gain>
+      <i_gain>0.0</i_gain>
+      <d_gain>1.0</d_gain>
+      <cmd_max>200.0</cmd_max>
+      <cmd_min>-200.0</cmd_min>
+    </plugin>
+  </gazebo>
+  <gazebo>
+    <plugin filename="gz-sim-joint-position-controller-system"
+            name="gz::sim::systems::JointPositionController">
+      <joint_name>armjoint_right</joint_name>
+      <topic>/armjoint_right/cmd_pos</topic>
+      <initial_position>0.0</initial_position>
+      <p_gain>20.0</p_gain>
+      <i_gain>0.0</i_gain>
+      <d_gain>1.0</d_gain>
+      <cmd_max>200.0</cmd_max>
+      <cmd_min>-200.0</cmd_min>
+    </plugin>
+  </gazebo>
   <gazebo>
     <plugin filename="gz-sim-odometry-publisher-system"

Commit message: Revert "Fix new_gazebo joint stability and add joint position controllers"
This reverts commit 2b2c9208486a072abbc8793870420e9407a78ff8.

File: ros2_ws/src/drobot_description/urdf_sub/drobotv0.urdf (robot description, URDF)
Before this commit: robot drobotv0, 11 links, 10 joints
Joints:
- removed joint wheeljoint_LF
- added joint wheejoint_LF: type continuous, parent arm_left, child wheel_LF, origin xyz=0.023562 0.08366 -0.059076 rpy=0 0 0, axis 0 0.99994 0.011086, limit lower=-3.14 upper=3.14 effort=1 velocity=1

File: ros2_ws/src/drobot_description/urdf_sub/drobotv0.urdf.xacro (robot description, xacro)
@@ -99,9 +99,8 @@
       xyz="1 0 0" />
     <limit
-      lower="-0.60"
-      upper="0.60"
-      effort="100"
-      velocity="2.0" />
-    <dynamics damping="40.0" friction="8.0" />
+      lower="-3.14"
+      upper="3.14"
+      effort="1"
+      velocity="1" />
   </joint>
   <link
@@ -158,9 +157,8 @@
       xyz="1 0 0" />
     <limit
-      lower="-0.40"
-      upper="0.90"
-      effort="120"
-      velocity="2.0" />
-    <dynamics damping="50.0" friction="10.0" />
+      lower="-3.14"
+      upper="3.14"
+      effort="1"
+      velocity="1" />
   </joint>
   <link
@@ -205,5 +203,5 @@
   </link>
   <joint
-    name="wheeljoint_LF"
+    name="wheejoint_LF"
     type="continuous">
     <origin
@@ -333,9 +331,12 @@
       xyz="-1 0 0" />
     <limit
-      lower="-0.60"
-      upper="0.60"
-      effort="100"
-      velocity="2.0" />
-    <dynamics damping="40.0" friction="8.0" />
+      lower="-3.14"
+      upper="3.14"
+      effort="1"
+      velocity="1" />
+    <mimic
+      joint="servo_LF"
+      multiplier="-1"
+      offset="0" />
   </joint>
   <link
@@ -392,9 +393,12 @@
       xyz="-1 0 0" />
     <limit
-      lower="-0.60"
-      upper="0.60"
-      effort="100"
-      velocity="2.0" />
-    <dynamics damping="40.0" friction="8.0" />
+      lower="-3.14"
+      upper="3.14"
+      effort="1"
+      velocity="1" />
+    <mimic
+      joint="servo_LF"
+      multiplier="1"
+      offset="0" />
   </joint>
   <link
@@ -451,9 +455,12 @@
       xyz="-1 0 0" />
     <limit
-      lower="-0.40"
-      upper="0.90"
-      effort="120"
-      velocity="2.0" />
-    <dynamics damping="50.0" friction="10.0" />
+      lower="-3.14"
+      upper="3.14"
+      effort="1"
+      velocity="1" />
+    <mimic
+      joint="armjoint_left"
+      multiplier="1"
+      offset="0" />
   </joint>
   <link
@@ -626,9 +633,12 @@
       xyz="1 0 0" />
     <limit
-      lower="-0.60"
-      upper="0.60"
-      effort="100"
-      velocity="2.0" />
-    <dynamics damping="40.0" friction="8.0" />
+      lower="-3.14"
+      upper="3.14"
+      effort="1"
+      velocity="1" />
+    <mimic
+      joint="servo_RF"
+      multiplier="-1"
+      offset="0" />
   </joint>
   <!-- Gazebo systems for teleop (/cmd_vel) -->
@@ -654,83 +664,4 @@
     </plugin>
   </gazebo>
-  <!-- Joint position controllers (Gazebo topic control) -->
-  <gazebo>
-    <plugin filename="gz-sim-joint-position-controller-system"
-            name="gz::sim::systems::JointPositionController">
-      <joint_name>servo_LF</joint_name>
-      <topic>/servo_LF/cmd_pos</topic>
-      <initial_position>0.0</initial_position>
-      <p_gain>20.0</p_gain>
-      <i_gain>0.0</i_gain>
-      <d_gain>1.0</d_gain>
-      <cmd_max>200.0</cmd_max>
-      <cmd_min>-200.0</cmd_min>
-    </plugin>
-  </gazebo>
-  <gazebo>
-    <plugin filename="gz-sim-joint-position-controller-system"
-            name="gz::sim::systems::JointPositionController">
-      <joint_name>servo_LR</joint_name>
-      <topic>/servo_LR/cmd_pos</topic>
-      <initial_position>0.0</initial_position>
-      <p_gain>20.0</p_gain>
-      <i_gain>0.0</i_gain>
-      <d_gain>1.0</d_gain>
-      <cmd_max>200.0</cmd_max>
-      <cmd_min>-200.0</cmd_min>
-    </plugin>
-  </gazebo>
-  <gazebo>
-    <plugin filename="gz-sim-joint-position-controller-system"
-            name="gz::sim::systems::JointPositionController">
-      <joint_name>servo_RF</joint_name>
-      <topic>/servo_RF/cmd_pos</topic>
-      <initial_position>0.0</initial_position>
-      <p_gain>20.0</p_gain>
-      <i_gain>0.0</i_gain>
-      <d_gain>1.0</d_gain>
-      <cmd_max>200.0</cmd_max>
-      <cmd_min>-200.0</cmd_min>
-    </plugin>
-  </gazebo>
-  <gazebo>
-    <plugin filename="gz-sim-joint-position-controller-system"
-            name="gz::sim::systems::JointPositionController">
-      <joint_name>servo_RR</joint_name>
-      <topic>/servo_RR/cmd_pos</topic>
-      <initial_position>0.0</initial_position>
-      <p_gain>20.0</p_gain>
-      <i_gain>0.0</i_gain>
-      <d_gain>1.0</d_gain>
-      <cmd_max>200.0</cmd_max>
-      <cmd_min>-200.0</cmd_min>
-    </plugin>
-  </gazebo>
-  <gazebo>
-    <plugin filename="gz-sim-joint-position-controller-system"
-            name="gz::sim::systems::JointPositionController">
-      <joint_name>armjoint_left</joint_name>
-      <topic>/armjoint_left/cmd_pos</topic>
-      <initial_position>0.0</initial_position>
-      <p_gain>20.0</p_gain>
-      <i_gain>0.0</i_gain>
-      <d_gain>1.0</d_gain>
-      <cmd_max>200.0</cmd_max>
-      <cmd_min>-200.0</cmd_min>
-    </plugin>
-  </gazebo>
-  <gazebo>
-    <plugin filename="gz-sim-joint-position-controller-system"
-            name="gz::sim::systems::JointPositionController">
-      <joint_name>armjoint_right</joint_name>
-      <topic>/armjoint_right/cmd_pos</topic>
-      <initial_position>0.0</initial_position>
-      <p_gain>20.0</p_gain>
-      <i_gain>0.0</i_gain>
-      <d_gain>1.0</d_gain>
-      <cmd_max>200.0</cmd_max>
-      <cmd_min>-200.0</cmd_min>
-    </plugin>
-  </gazebo>
   <gazebo>
     <plugin filename="gz-sim-odometry-publisher-system"
